File: BenchBudEE.kicad_pcb (KiCad board)
At the start: 4 copper layers, 165.1 x 63.5 mm, 109 parts, among them K1 RELAY, P1 24 Pin MiniFit JR, P2 CONN_2, P3 CONN_3X2, P4 12 Pin Terminal Block, P5 CONN_3, Q1 2N3904, Q2 MOSFET_N, Q3 NMOS, Q4 NMOS, SW1 SWITCH, U1 OPTO_TRANSISTOR, U10 LM317K, U2 MCP3901, U3 LMT84, U4 OPA4170, U5 AP5726, U6 MCP4801, U7 LM337T, U8 LM317K, U9 LM337T

Commit message: Layout v3.0
Parts:
- added V8508H: VAL**, V8508H, F.Cu at (171.8, 138.5)
- added V8508H: VAL**, V8508H, F.Cu at (185.9, 138.5)
- moved R35 58.1 mm to (112.3, 122.9)
- moved R49 57.7 mm to (113.5, 128.4)
- moved C16 57.7 mm to (109.8, 128.3)
- moved R48 57.7 mm to (113.6, 125.7)
- moved R37 55.5 mm to (129.6, 122.7)
- moved C17 48.6 mm to (173.1, 126.9)
- moved R51 48.6 mm to (169.2, 126.9)
- moved C15 48.6 mm to (175.4, 129.4)
- moved R39 48.6 mm to (169.1, 124.4)
- moved R50 48.6 mm to (171.1, 129.3)
- moved C14 44.5 mm to (139.6, 123.0)
- moved R36 44.5 mm to (143.3, 123.1)
- moved C19 44.5 mm to (143.2, 127.8)
- moved R40 44.5 mm to (143.2, 125.4)
- moved R41 44.5 mm to (139.6, 125.4)
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Changed lines of the file:
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@@
     (links 288)
     (no_connects 250)
-    (area 63.190199 104.582599 232.434601 184.889)
+    (area 63.190199 99.527999 232.434601 184.889)
     (thickness 1.6)
     (drawings 4)
     (tracks 0)
     (zones 0)
-    (modules 109)
+    (modules 111)
     (nets 96)
   )
@@
     (mod_text_size 1 1)
     (mod_text_width 0.15)
-    (pad_size 3.175 3.175)
-    (pad_drill 3.175)
+    (pad_size 2.5 2.5)
+    (pad_drill 1.5)
     (pad_to_mask_clearance 0.254)
     (solder_mask_min_width 0.127)
@@
   )
   (module SMA (layer F.Cu)
-    (at 219.8116 142.4432 90)
+    (at 219.202 151.8031 90)
     (fp_text reference D5 (at 0 -2.54 90) (layer F.SilkS)
       (effects (font (size 1 1) (thickness 0.15)))
@@
   )
   (module SM1812 (layer F.Cu)
-    (at 217.8812 133.9977)
+    (at 217.2716 143.3576)
     (tags "CMS SM")
     (attr smd)
@@
   )
   (module SM1206 (layer B.Cu)
-    (at 197.9803 140.2969)
+    (at 197.3707 149.6568)
     (attr smd)
     (fp_text reference R33 (at 0 0) (layer B.SilkS)
@@
   )
   (module SM0805 (layer F.Cu)
-    (at 213.2457 134.3025 270)
+    (at 212.6361 143.6624 270)
     (attr smd)
     (fp_text reference C13 (at 0 -0.3175 270) (layer F.SilkS)
@@
   )
   (module DPAK2 (layer F.Cu)
-    (at 214.6554 140.5763 90)
+    (at 214.0458 149.9362 90)
     (descr "MOS boitier DPACK G-D-S")
     (tags "CMD DPACK")
@@
   )
   (module DPAK2 (layer F.Cu)
-    (at 199.5551 140.5763 90)
+    (at 198.9455 149.9362 90)
     (descr "MOS boitier DPACK G-D-S")
     (tags "CMD DPACK")
@@
   )
   (module SM0805 (layer B.Cu)
-    (at 103.5304 122.4788 180)
+    (at 96.3422 126.1237 180)
     (attr smd)
     (fp_text reference R30 (at 0 0.3175 180) (layer B.SilkS)
@@
   )
   (module SPDT_SW (layer F.Cu)
-    (at 102.5144 124.5616 180)
+    (at 95.2754 124.1806 180)
     (fp_text reference SW1 (at 0.325 -3 180) (layer F.SilkS)
       (effects (font (size 1 1) (thickness 0.15)))
@@
   )
   (module SM0805 (layer B.Cu)
-    (at 126.7841 127.9525)
+    (at 175.4124 129.3749)
     (attr smd)
     (fp_text reference C15 (at 0 0.3175) (layer B.SilkS)
@@
   )
   (module SM0805 (layer B.Cu)
-    (at 182.9943 132.9182 180)
+    (at 139.6111 123.0122 180)
     (attr smd)
     (fp_text reference C14 (at 0 0.3175 180) (layer B.SilkS)
@@
   )
   (module SM0805 (layer B.Cu)
-    (at 186.6138 137.7061 180)
+    (at 143.2306 127.8001 180)
     (attr smd)
     (fp_text reference C19 (at 0 0.3175 180) (layer B.SilkS)
@@
   )
   (module SM0805 (layer B.Cu)
-    (at 167.2336 133.8834)
+    (at 109.8296 128.3208)
     (attr smd)
     (fp_text reference C16 (at 0 0.3175) (layer B.SilkS)
@@
   )
   (module SM0805 (layer B.Cu)
-    (at 124.4473 125.5141)
+    (at 173.0756 126.9365)
     (attr smd)
     (fp_text reference C17 (at 0 0.3175) (layer B.SilkS)
@@
   )
   (module SM0805 (layer B.Cu)
-    (at 157.5435 123.8377 180)
+    (at 183.8198 125.1331 180)
     (attr smd)
     (fp_text reference C18 (at 0 0.3175 180) (layer B.SilkS)
@@
   )
   (module SM0805 (layer B.Cu)
-    (at 170.9801 131.2545 180)
+    (at 113.5761 125.6919 180)
     (attr smd)
     (fp_text reference R48 (at 0 0.3175 180) (layer B.SilkS)
@@
   )
   (module SM0805 (layer B.Cu)
-    (at 170.942 133.9596)
+    (at 113.538 128.397)
     (attr smd)
     (fp_text reference R49 (at 0 0.3175) (layer B.SilkS)
@@
   )
   (module SM0805 (layer B.Cu)
-    (at 120.5611 125.4379 180)
+    (at 169.1894 126.8603 180)
     (attr smd)
     (fp_text reference R51 (at 0 0.3175 180) (layer B.SilkS)
@@
   )
   (module SM0805 (layer B.Cu)
-    (at 122.4407 127.8509 180)
+    (at 171.069 129.2733 180)
     (attr smd)
     (fp_text reference R50 (at 0 0.3175 180) (layer B.SilkS)
@@
   )
   (module SM0805 (layer B.Cu)
-    (at 186.6138 135.3312)
+    (at 143.2306 125.4252)
     (attr smd)
     (fp_text reference R40 (at 0 0.3175) (layer B.SilkS)
@@
   )
   (module SM0805 (layer B.Cu)
-    (at 183.0324 135.3312)
+    (at 139.6492 125.4252)
     (attr smd)
     (fp_text reference R41 (at 0 0.3175) (layer B.SilkS)
@@
   )
   (module SM0805 (layer B.Cu)
-    (at 120.4341 122.9487 180)
+    (at 169.0624 124.3711 180)
     (attr smd)
     (fp_text reference R39 (at 0 0.3175 180) (layer B.SilkS)
@@
   )
   (module SM0805 (layer B.Cu)
-    (at 161.671 127.5969)
+    (at 187.9473 128.8923)
     (attr smd)
     (fp_text reference R38 (at 0 0.3175) (layer B.SilkS)
@@
   )
   (module SM0805 (layer B.Cu)
-    (at 161.2773 123.7615)
+    (at 187.5536 125.0569)
     (attr smd)
     (fp_text reference R34 (at 0 0.3175) (layer B.SilkS)
@@
   )
   (module SM0805 (layer B.Cu)
-    (at 186.6646 132.9817 180)
+    (at 143.2814 123.0757 180)
     (attr smd)
     (fp_text reference R36 (at 0 0.3175 180) (layer B.SilkS)
@@
   )
   (module POT_EVUE3K (layer F.Cu)
-    (at 184.8358 127.7366 90)
+    (at 129.6162 122.682 90)
     (fp_text reference R37 (at 0.075 -7.15 90) (layer F.SilkS)
       (effects (font (size 1 1) (thickness 0.15)))
@@
   )
   (module POT_EVUE3K (layer F.Cu)
-    (at 170.2054 127.7366 90)
+    (at 112.268 122.936 90)
     (fp_text reference R35 (at 0.075 -7.15 90) (layer F.SilkS)
       (effects (font (size 1 1) (thickness 0.15)))
@@
   )
   (module TO220_VERT (layer F.Cu)
-    (at 136.652 125.349 90)
+    (at 171.9707 134.6327 90)
     (descr "Regulateur TO220 serie LM78xx")
     (tags "TR TO220")
-    (fp_text reference U8 (at -3.175 0 180) (layer F.SilkS)
+    (fp_text reference U8 (at 3.683 -3.9497 180) (layer F.SilkS)
       (effects (font (size 1.524 1.016) (thickness 0.2032)))
     )
-    (fp_text value LM317K (at 0.635 -6.35 90) (layer F.SilkS)
+    (fp_text value LM317K (at 0.635 -6.35 90) (layer F.SilkS) hide
       (effects (font (size 1.524 1.016) (thickness 0.2032)))
     )
@@
   )
   (module TO220_VERT (layer F.Cu)
-    (at 150.4315 125.1966 90)
+    (at 185.8899 134.8613 90)
     (descr "Regulateur TO220 serie LM78xx")
     (tags "TR TO220")
-    (fp_text reference U10 (at -3.175 0 180) (layer F.SilkS)
+    (fp_text reference U10 (at 3.556 -3.556 180) (layer F.SilkS)
       (effects (font (size 1.524 1.016) (thickness 0.2032)))
     )
-    (fp_text value LM317K (at 0.635 -6.35 90) (layer F.SilkS)
+    (fp_text value LM317K (at 0.635 -6.35 90) (layer F.SilkS) hide
       (effects (font (size 1.524 1.016) (thickness 0.2032)))
     )
@@
   )
   (module TO220_VERT (layer F.Cu)
-    (at 198.1454 127.7366 90)
+    (at 202.9587 132.7658 90)
     (descr "Regulateur TO220 serie LM78xx")
     (tags "TR TO220")
@@
   )
   (module TO220_VERT (layer F.Cu)
-    (at 210.3374 127.4064 90)
+    (at 202.946 125.603 90)
     (descr "Regulateur TO220 serie LM78xx")
     (tags "TR TO220")
@@
       (layers *.Cu *.Mask F.SilkS)
     )
+  )
+  (module V8508H (layer F.Cu)
+    (at 171.8437 138.5062 180)
+    (fp_text reference V8508H (at -3.4 11.8 180) (layer F.SilkS)
+      (effects (font (size 1 1) (thickness 0.15)))
+    )
+    (fp_text value VAL** (at 4.35 11.95 180) (layer F.SilkS) hide
+      (effects (font (size 1 1) (thickness 0.15)))
+    )
+    (fp_line (start 0 0) (end 6.4 0) (layer F.SilkS) (width 0.15))
+    (fp_line (start 6.4 0) (end 6.4 12.7) (layer F.SilkS) (width 0.15))
+    (fp_line (start 6.4 12.7) (end -6.4 12.7) (layer F.SilkS) (width 0.15))
+    (fp_line (start -6.4 12.7) (end -6.4 0) (layer F.SilkS) (width 0.15))
+    (fp_line (start -6.4 0) (end 0 0) (layer F.SilkS) (width 0.15))
+    (pad 1 thru_hole circle (at 0 0 180) (size 2.5 2.5) (drill 1.5)
+      (layers *.Cu *.Mask F.SilkS)
+    )
+  )
+  (module V8508H (layer F.Cu)
+    (at 185.8899 138.5062 180)
+    (fp_text reference V8508H (at -3.4 11.8 180) (layer F.SilkS)
+      (effects (font (size 1 1) (thickness 0.15)))
+    )
+    (fp_text value VAL** (at 4.35 11.95 180) (layer F.SilkS) hide
+      (effects (font (size 1 1) (thickness 0.15)))
+    )
+    (fp_line (start 0 0) (end 6.4 0) (layer F.SilkS) (width 0.15))
+    (fp_line (start 6.4 0) (end 6.4 12.7) (layer F.SilkS) (width 0.15))
+    (fp_line (start 6.4 12.7) (end -6.4 12.7) (layer F.SilkS) (width 0.15))
+    (fp_line (start -6.4 12.7) (end -6.4 0) (layer F.SilkS) (width 0.15))
+    (fp_line (start -6.4 0) (end 0 0) (layer F.SilkS) (width 0.15))
+    (pad 1 thru_hole circle (at 0 0 180) (size 2.5 2.5) (drill 1.5)
+      (layers *.Cu *.Mask F.SilkS)
+    )
