File: BenchBudEE.kicad_pcb (KiCad board)
At the start: 4 copper layers, 165.1 x 63.5 mm, 118 parts, among them K1 RELAY, P1 24 Pin MiniFit JR, P2 CONN_2, P3 CONN_3X2, P4 12 Pin Terminal Block, P5 CONN_3, Q1 2N3904, Q2 MOSFET_N, Q3 NMOS, Q4 NMOS, SW1 SWITCH, U1 OPTO_TRANSISTOR, U10 LM317K, U2 MCP3901, U3 LMT84, U4 OPA4170, U5 AP5726, U6 MCP4801, U7 LM337T, U8 LM317K, U9 LM337T

Commit message: Layout v13.0
Parts:
- added C22: C, SM1210, B.Cu at (222.9, 137.0)
- added C23: C, SM1210, F.Cu at (222.8, 133.2)
- added C24: C, SM1210, B.Cu at (222.2, 128.5)
- added C25: C, SM1210, B.Cu at (222.2, 124.7)
- added R52: R, SM0805, B.Cu at (228.7, 155.1)
- R10, R11, R12, R13, R14, R15, R16, R17, R18, R19, R20, R21, R42, R43, R46, R47, R7, R8, R9: footprint SM0805-bridge -> SM0805-BR
Routing:
- net GND_PWR: track 12.6 -> 49.7 mm, vias 4 -> 5
- net +12V: track 128.4 -> 132.0 mm
- net +3.3V: track 151.0 -> 154.4 mm
- net +5V: track 73.8 -> 77.1 mm
- net N-0000084: track 0.00 -> 3.18 mm
- net /Fan/TACH: track 94.4 -> 97.1 mm
- net /Power_Adjustment_Monitor/V-_ADJ: track 73.5 -> 76.1 mm
- net /Power_Adjustment_Monitor/V+_ADJ: track 53.1 -> 55.7 mm

Commit message: Layout v14.0
Parts:
- added C26: C, SM0805, B.Cu at (170.5, 149.7)
- added C27: C, SM0805, B.Cu at (167.4, 142.5)
Connections:
- U2 pad 10: (no net) -> N-0000067
- U2 pad 15: (no net) -> N-0000070
- U2 pad 16: (no net) -> N-0000068
- U2 pad 9: (no net) -> N-0000071
Routing:
- net +12C: track 207.4 -> 202.3 mm
- net N-0000068: track 0.00 -> 4.78 mm, vias 0 -> 1
- net N-0000070: track 0.00 -> 4.47 mm, vias 0 -> 1
- net N-0000067: track 0.00 -> 2.85 mm, vias 0 -> 1
- net N-0000071: track 0.00 -> 2.80 mm, vias 0 -> 1
- net GND_LED: track 11.7 -> 9.71 mm, vias 3 -> 2
Other:
- net class Default: clearance 0.254 -> 0.1524
- rule pad_to_mask_clearance: 0.254 -> 0.0762
- rule solder_mask_min_width: 0.127 -> 0.0508
- rule trace_clearance: 0.254 -> 0.1524

Commit message: Layout v15.0
Parts:
- added G***: LOGO, LOGO, F.Cu at (115.7, 174.2)
- D2, R5: moved to F.Cu
- moved D2 13.4 mm to (194.6, 176.3)
- moved R5 9.29 mm to (193.8, 168.7)
- moved D1 7.54 mm to (186.9, 177.0)
- moved Q1 7.54 mm to (189.9, 182.0)
- moved R1 7.54 mm to (176.2, 174.0)
- moved R2 7.54 mm to (185.2, 178.9)
- moved R3 7.54 mm to (190.4, 178.0)
- moved R4 7.54 mm to (189.9, 168.7)
- moved R6 7.54 mm to (185.1, 181.5)
- moved U1 7.54 mm to (179.8, 171.4)
Routing:
- net /Arduino/RELAY-: track 46.7 -> 39.2 mm
- net /Arduino/RELAY+: track 67.7 -> 60.2 mm
- net N-0000088: track 14.0 -> 20.0 mm
- net N-0000092: track 7.07 -> 12.6 mm
- net GND_LED: track 9.71 -> 11.5 mm, vias 2 -> 3
- net GND_RELAY: track 5.79 -> 4.37 mm
- net +12P: track 71.2 -> 70.1 mm
Other:
- net class AC added: clearance 1.524, trace_width 3.81, via_dia 1.1684, via_drill 0.6096

Commit message: Layout v16.0
Parts:
- added TP10: FE_V-, TP_TH, F.Cu at (210.6, 126.6)
- added TP11: AGND, TP_TH, F.Cu at (209.2, 141.5)
- added TP2: +5V, TP_TH, F.Cu at (162.8, 141.0)
- added TP3: CH0+, TP_TH, F.Cu at (161.3, 134.8)
- added TP4: CH1+, TP_TH, F.Cu at (215.4, 144.7)
- added TP5: DAC_OUT, TP_TH, F.Cu at (180.7, 151.2)
- added TP6: +12P, TP_TH, F.Cu at (188.8, 164.7)
- added TP7: RLY-, TP_TH, F.Cu at (179.5, 182.8)
- added TP8: GND_PWR, TP_TH, F.Cu at (192.5, 127.5)
- added TP9: FE_V+, TP_TH, F.Cu at (200.1, 127.6)
- Q3, Q4: footprint DPAK2 -> DPAK2_NO
- U10, U8: value LM317K -> LM317T; footprint TO220_VERT -> TO220_VERT1
- U7, U9: footprint TO220_VERT -> TO220_VERT1
- moved U8 20.2 mm to (183.6, 126.9), turned to 270 degrees
- moved U10 20.0 mm to (201.3, 136.3), turned to 90 degrees
- moved C14 9.56 mm to (165.5, 123.6), turned to 180 degrees
- moved R49 6.92 mm to (219.9, 133.9), turned to 270 degrees
- moved R41 6.52 mm to (171.4, 133.0), turned to 180 degrees
- moved C19 4.04 mm to (172.5, 130.2), turned to 270 degrees
- moved C11 3.65 mm to (212.7, 139.6), turned to 180 degrees
- moved C21 2.92 mm to (212.7, 141.6), turned to 0 degrees
- moved R40 2.26 mm to (170.1, 130.2), turned to 90 degrees
- moved R36 1.48 mm to (164.9, 127.8), turned to 90 degrees
- moved U7 0.20 mm to (213.5, 136.4)
- moved U9 0.17 mm to (169.8, 127.0)
Connections:
- R34 pad 2: N-00000122 (its old number) -> N-00000121
- R35 pad 1: N-00000122 (its old number) -> N-00000121
- U10 pad 1: N-00000122 (its old number) -> N-00000123
- U10 pad 2: +12V -> FE_V+
- U10 pad 3: /Power_Adjustment_Monitor/V+_ADJ -> +12V
- U8 pad 1: N-00000123 -> N-00000121
- U8 pad 2: +12V -> /Power_Adjustment_Monitor/V+_ADJ
- U8 pad 3: FE_V+ -> +12V
Routing:
- net N-00000122 (its old number): track 73.6 -> 0.00 mm
- net N-00000121: track 0.00 -> 73.6 mm
- net FE_V-: track 35.7 -> 51.7 mm
- net N-0000091: track 20.0 -> 30.9 mm
- net FE_V+: track 36.8 -> 46.6 mm
- net +5V: track 77.1 -> 86.9 mm
- net N-0000072: track 29.2 -> 35.7 mm
- net GND_PWR: track 49.7 -> 55.0 mm, vias 5 -> 4
- net -12V: track 136.4 -> 141.4 mm
- net +12P: track 70.1 -> 75.1 mm
- net +3.3V: track 154.4 -> 150.4 mm, vias 0 -> 1
- net N-00000119: track 7.42 -> 11.4 mm
- net /Arduino/V-_ADJ_MON: track 119.9 -> 123.6 mm, vias 2 -> 0
- net N-0000071: track 56.7 -> 58.8 mm
- net /Arduino/~RESET: track 32.6 -> 34.6 mm
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
Commit message: Layout v17.0
Parts:
- added C28: C, SM0805, F.Cu at (182.8, 155.3)
- added R53: 1k, SM0805, F.Cu at (211.3, 144.9)
- added R54: 1k, SM0805, B.Cu at (217.4, 147.7)
- added R55: 0, SM0805, B.Cu at (202.3, 151.1)
- moved R33 1.30 mm to (182.9, 159.3)
- moved TP5 0.40 mm to (180.3, 151.1)
Connections:
- P4 pad 6: /Terminal_Block/TC_IN_+ -> /Terminal_Block/TC_IN_-
- P4 pad 7: /Terminal_Block/TC_IN_- -> /Terminal_Block/TC_IN_+
- Q3 pad 2: /Arduino/CURR_MEAS -> N-00000120
- Q4 pad 1: N-00000118 (its old number) -> N-00000119
- Q4 pad 3: /Arduino/CURR_MEAS -> N-00000120
- R33 pad 1: /Arduino/CURR_MEAS -> N-00000120
- TP4 pad 1: N-0000071 (its old number) -> N-0000069
- U2 pad 7: N-0000071 (its old number) -> N-0000069
- U3 pad 3: N-0000071 (its old number) -> N-0000070
- U4 pad 10: /Terminal_Block/TC_IN_+ -> /Terminal_Block/TC_IN_-
- U4 pad 12: /Terminal_Block/TC_IN_- -> /Terminal_Block/TC_IN_+
- U4 pad 7: N-00000118 (its old number) -> N-00000120
Routing:
- net N-0000069: track 0.00 -> 59.3 mm, vias 0 -> 1
- net N-0000071 (its old number): track 58.8 -> 0.00 mm, vias 1 -> 0
- net N-00000120: track 0.00 -> 54.2 mm, vias 0 -> 3
- net N-00000118 (its old number): track 25.9 -> 0.00 mm
- net /Arduino/CURR_MEAS: track 77.8 -> 58.9 mm
- net AGND: track 64.7 -> 69.1 mm
- net N-00000119: track 0.00 -> 4.06 mm, vias 0 -> 1
- net /Terminal_Block/TC_IN_-: track 44.9 -> 41.8 mm
- net /Terminal_Block/TC_IN_+: track 41.8 -> 44.9 mm
- net N-0000070: track 0.00 -> 1.74 mm
- added copper zone on F.Cu, net N-00000120
- removed copper zone on F.Cu, net /Arduino/CURR_MEAS

Commit message: Layout v17.1
Parts:
- moved TP5 1.00 mm to (181.1, 151.8)
- moved C28 0.89 mm to (181.9, 155.2), turned to 180 degrees
Connections:
- Q3 pad 2: N-00000120 -> /Arduino/CURR_MEAS
- Q4 pad 3: N-00000120 -> /Arduino/CURR_MEAS
- R33 pad 1: N-00000120 -> /Arduino/CURR_MEAS
Routing:
- net N-00000120: track 54.2 -> 25.7 mm, vias 3 -> 1
- net /Arduino/CURR_MEAS: track 58.9 -> 71.0 mm
- net N-00000121: track 11.4 -> 12.5 mm
- added copper zone on F.Cu, net /Arduino/CURR_MEAS
- removed copper zone on F.Cu, net N-00000120
Changed lines of the file:
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@@
     (thickness 1.6)
     (drawings 4)
-    (tracks 889)
+    (tracks 883)
     (zones 0)
     (modules 140)
@@
     (pad 3 smd rect (at 2.286 0 180) (size 1.651 3.048)
       (layers F.Cu F.Paste F.Mask)
-      (net 50 N-00000120)
+      (net 9 /Arduino/CURR_MEAS)
     )
     (model smd/dpack_2.wrl
@@
     (pad 2 smd rect (at 0 -6.35 180) (size 6.096 6.096)
       (layers F.Cu F.Paste F.Mask)
-      (net 50 N-00000120)
+      (net 9 /Arduino/CURR_MEAS)
     )
     (pad 3 smd rect (at 2.286 0 180) (size 1.651 3.048)
@@
     (pad 1 smd rect (at -1.651 0) (size 1.524 2.032)
       (layers F.Cu F.Paste F.Mask)
-      (net 50 N-00000120)
+      (net 9 /Arduino/CURR_MEAS)
     )
     (pad 2 smd rect (at 1.651 0) (size 1.524 2.032)
@@
   )
   (module TP_TH (layer F.Cu)
-    (at 180.3273 151.1046)
+    (at 181.08676 151.75738)
     (fp_text reference TP5 (at 0.5842 1.9304) (layer F.SilkS)
       (effects (font (size 0.635 0.635) (thickness 0.127)))
@@
   )
   (module SM0805 (layer F.Cu)
-    (at 182.8038 155.2956)
+    (at 181.9148 155.2194 180)
     (attr smd)
-    (fp_text reference C28 (at -0.51816 -1.16078) (layer F.SilkS)
+    (fp_text reference C28 (at -0.51816 -1.16078 180) (layer F.SilkS)
       (effects (font (size 0.50038 0.50038) (thickness 0.10922)))
     )
-    (fp_text value C (at 0 0.381) (layer F.SilkS) hide
+    (fp_text value C (at 0 0.381 180) (layer F.SilkS) hide
       (effects (font (size 0.50038 0.50038) (thickness 0.10922)))
     )
@@
     (fp_line (start 1.524 -0.762) (end 1.524 0.762) (layer F.SilkS) (width 0.09906))
     (fp_line (start 1.524 0.762) (end 0.508 0.762) (layer F.SilkS) (width 0.09906))
-    (pad 1 smd rect (at -0.9525 0) (size 0.889 1.397)
+    (pad 1 smd rect (at -0.9525 0 180) (size 0.889 1.397)
       (layers F.Cu F.Paste F.Mask)
       (net 50 N-00000120)
     )
-    (pad 2 smd rect (at 0.9525 0) (size 0.889 1.397)
+    (pad 2 smd rect (at 0.9525 0 180) (size 0.889 1.397)
       (layers F.Cu F.Paste F.Mask)
       (net 9 /Arduino/CURR_MEAS)
@@
   (segment (start 169.799 125.222) (end 170.815 125.222) (width 0.9144) (layer PWR) (net 8))
   (segment (start 96.393 128.016) (end 99.06 128.016) (width 0.9144) (layer F.Cu) (net 8))
-  (via (at 182.55996 164.90188) (size 0.508) (drill 0.3302) (layers F.Cu B.Cu) (net 9))
-  (segment (start 150.241 169.72788) (end 155.067 164.90188) (width 0.254) (layer B.Cu) (net 9))
-  (segment (start 155.067 164.90188) (end 182.55996 164.90188) (width 0.254) (layer B.Cu) (net 9))
+  (segment (start 182.16499 147.78863) (end 181.21757 147.78863) (width 0.254) (layer F.Cu) (net 9))
+  (segment (start 179.2986 149.7076) (end 179.2986 153.6192) (width 0.254) (layer F.Cu) (net 9))
+  (segment (start 181.21757 147.78863) (end 179.2986 149.7076) (width 0.254) (layer F.Cu) (net 9))
+  (segment (start 180.9623 155.2194) (end 179.6034 155.2194) (width 0.254) (layer F.Cu) (net 9))
+  (segment (start 179.6034 155.2194) (end 179.4764 155.0924) (width 0.254) (layer F.Cu) (net 9))
   (segment (start 150.241 175.5775) (end 150.241 169.72788) (width 0.254) (layer B.Cu) (net 9))
-  (segment (start 183.7563 156.591) (end 183.7563 155.2956) (width 0.254) (layer F.Cu) (net 9))
-  (segment (start 183.0324 157.3149) (end 183.7563 156.591) (width 0.254) (layer F.Cu) (net 9))
-  (segment (start 183.0324 164.42944) (end 183.0324 157.3149) (width 0.254) (layer F.Cu) (net 9))
-  (segment (start 182.55996 164.90188) (end 183.0324 164.42944) (width 0.254) (layer F.Cu) (net 9))
-  (segment (start 182.16499 147.78863) (end 182.99303 147.78863) (width 0.254) (layer F.Cu) (net 9))
-  (segment (start 182.99303 147.78863) (end 183.24576 148.04136) (width 0.254) (layer F.Cu) (net 9))
-  (segment (start 183.24576 148.04136) (end 183.24576 154.78506) (width 0.254) (layer F.Cu) (net 9))
-  (segment (start 183.24576 154.78506) (end 183.7563 155.2956) (width 0.254) (layer F.Cu) (net 9))
+  (segment (start 165.85184 165.01364) (end 165.85184 160.43148) (width 0.254) (layer F.Cu) (net 9))
+  (segment (start 165.57244 165.29304) (end 165.85184 165.01364) (width 0.254) (layer F.Cu) (net 9))
+  (via (at 165.57244 165.29304) (size 0.508) (drill 0.3302) (layers F.Cu B.Cu) (net 9))
+  (segment (start 154.67584 165.29304) (end 165.57244 165.29304) (width 0.254) (layer B.Cu) (net 9))
+  (segment (start 150.241 169.72788) (end 154.67584 165.29304) (width 0.254) (layer B.Cu) (net 9))
+  (segment (start 200.1774 152.4) (end 191.5414 152.4) (width 0.254) (layer F.Cu) (net 9))
+  (segment (start 186.80684 157.13456) (end 178.92776 157.13456) (width 0.254) (layer F.Cu) (net 9))
+  (segment (start 191.5414 152.4) (end 186.80684 157.13456) (width 0.254) (layer F.Cu) (net 9))
+  (segment (start 181.2925 159.3342) (end 174.38624 159.3342) (width 0.6096) (layer F.Cu) (net 9))
+  (segment (start 174.38624 159.3342) (end 171.71924 156.6672) (width 0.254) (layer F.Cu) (net 9))
   (segment (start 174.00524 150.3172) (end 174.00524 142.14856) (width 0.254) (layer F.Cu) (net 10))
   (segment (start 159.0929 138.1887) (end 157.9118 138.1887) (width 0.254) (layer F.Cu) (net 10))
@@
   (via (at 203.1365 153.2128) (size 0.508) (drill 0.3302) (layers F.Cu B.Cu) (net 49))
   (segment (start 203.2254 153.1239) (end 203.1365 153.2128) (width 0.254) (layer B.Cu) (net 49))
-  (segment (start 181.8513 155.2956) (end 181.8513 156.7434) (width 0.254) (layer F.Cu) (net 50))
-  (segment (start 184.9247 156.9085) (end 184.9247 156.6545) (width 0.254) (layer F.Cu) (net 50))
-  (segment (start 184.8231 157.0101) (end 184.9247 156.9085) (width 0.254) (layer F.Cu) (net 50))
-  (via (at 184.8231 157.0101) (size 0.508) (drill 0.3302) (layers F.Cu B.Cu) (net 50))
-  (segment (start 181.737 157.0101) (end 184.8231 157.0101) (width 0.254) (layer B.Cu) (net 50))
-  (segment (start 181.6608 156.9339) (end 181.737 157.0101) (width 0.254) (layer B.Cu) (net 50))
-  (via (at 181.6608 156.9339) (size 0.508) (drill 0.3302) (layers F.Cu B.Cu) (net 50))
-  (segment (start 181.8513 156.7434) (end 181.6608 156.9339) (width 0.254) (layer F.Cu) (net 50))
-  (segment (start 181.8513 155.2956) (end 173.09084 155.2956) (width 0.254) (layer F.Cu) (net 50))
-  (segment (start 173.09084 155.2956) (end 171.71924 156.6672) (width 0.254) (layer F.Cu) (net 50))
-  (segment (start 182.16499 149.05863) (end 182.16499 154.98191) (width 0.254) (layer F.Cu) (net 50))
-  (segment (start 182.16499 154.98191) (end 181.8513 155.2956) (width 0.254) (layer F.Cu) (net 50))
-  (segment (start 200.1774 152.4) (end 189.1792 152.4) (width 0.254) (layer F.Cu) (net 50))
-  (segment (start 189.1792 152.4) (end 184.9247 156.6545) (width 0.254) (layer F.Cu) (net 50))
-  (segment (start 184.9247 156.6545) (end 184.912 156.6672) (width 0.254) (layer F.Cu) (net 50))
-  (segment (start 181.2925 159.3342) (end 174.38624 159.3342) (width 0.6096) (layer F.Cu) (net 50))
-  (segment (start 174.38624 159.3342) (end 171.71924 156.6672) (width 0.254) (layer F.Cu) (net 50))
-  (segment (start 200.1774 152.4) (end 200.7997 152.4) (width 0.254) (layer F.Cu) (net 50))
-  (segment (start 200.7997 152.4) (end 201.676 153.2763) (width 0.254) (layer F.Cu) (net 50))
-  (via (at 201.676 153.2763) (size 0.508) (drill 0.3302) (layers F.Cu B.Cu) (net 50))
-  (segment (start 201.676 153.2763) (end 201.3204 152.9207) (width 0.254) (layer B.Cu) (net 50))
-  (segment (start 201.3204 152.9207) (end 201.3204 151.1427) (width 0.254) (layer B.Cu) (net 50))
-  (segment (start 180.3273 151.1046) (end 180.3273 150.3807) (width 0.254) (layer B.Cu) (net 51))
-  (segment (start 178.7271 148.7805) (end 177.6984 148.7805) (width 0.254) (layer B.Cu) (net 51))
-  (segment (start 180.3273 150.3807) (end 178.7271 148.7805) (width 0.254) (layer B.Cu) (net 51))
+  (segment (start 182.8673 155.2194) (end 182.8673 153.0731) (width 0.254) (layer F.Cu) (net 50))
+  (segment (start 183.18988 152.75052) (end 183.18988 149.92858) (width 0.254) (layer F.Cu) (net 50))
+  (segment (start 182.8673 153.0731) (end 183.18988 152.75052) (width 0.254) (layer F.Cu) (net 50))
+  (segment (start 182.16499 149.05863) (end 182.31993 149.05863) (width 0.254) (layer F.Cu) (net 50))
+  (segment (start 197.0913 151.1427) (end 201.3204 151.1427) (width 0.254) (layer B.Cu) (net 50))
+  (segment (start 196.7484 151.4856) (end 197.0913 151.1427) (width 0.254) (layer B.Cu) (net 50))
+  (via (at 196.7484 151.4856) (size 0.508) (drill 0.3302) (layers F.Cu B.Cu) (net 50))
+  (segment (start 187.4901 151.4856) (end 196.7484 151.4856) (width 0.254) (layer F.Cu) (net 50))
+  (segment (start 186.9948 150.9903) (end 187.4901 151.4856) (width 0.254) (layer F.Cu) (net 50))
+  (segment (start 184.2516 150.9903) (end 186.9948 150.9903) (width 0.254) (layer F.Cu) (net 50))
+  (segment (start 182.31993 149.05863) (end 183.18988 149.92858) (width 0.254) (layer F.Cu) (net 50))
+  (segment (start 183.18988 149.92858) (end 184.2516 150.9903) (width 0.254) (layer F.Cu) (net 50))
+  (segment (start 181.08676 151.75738) (end 181.08676 151.003) (width 0.254) (layer B.Cu) (net 51))
+  (segment (start 178.86426 148.7805) (end 177.6984 148.7805) (width 0.254) (layer B.Cu) (net 51))
+  (segment (start 181.08676 151.003) (end 178.86426 148.7805) (width 0.254) (layer B.Cu) (net 51))
   (segment (start 177.6984 148.7805) (end 177.6984 147.18538) (width 0.254) (layer B.Cu) (net 51))
   (segment (start 177.6984 147.18538) (end 177.19802 146.685) (width 0.254) (layer B.Cu) (net 51))
@@
     )
   )
-  (zone (net 50) (net_name N-00000120) (layer F.Cu) (hatch edge 0.508)
+  (zone (net 9) (net_name /Arduino/CURR_MEAS) (layer F.Cu) (hatch edge 0.508)
     (connect_pads thru_hole_only (clearance 0.508))
     (min_thickness 0.254)

Commit message: Layout 18.0
Parts:
- JP1, JP2, JP3, JP4: footprint GND_PNT -> GND_PNT_1
- moved JP2 2.89 mm to (117.8, 167.7), turned to 270 degrees
- moved JP1 1.91 mm to (125.0, 155.4)
Routing:
- net GND: track 104.5 -> 39.4 mm
- net +5P: track 50.4 -> 54.2 mm
Other:
- rule via_min_size: 0.508 -> 0.6858

Commit message: Layout v19.0
Parts:
- removed TP1: CONN_1, 1pin
