File: Fan.sch (KiCad schematic (older format))
At the start: 11 parts, among them Q2 MOSFET_N, Q3 NMOS, Q4 NMOS, U4 OPA4170, U6 MCP4801

Commit message: Layout v5.0
Connections:
- net GND_FAN renamed AGND
Changed lines of the file:
@@
 Sheet 6 9
 Title ""
-Date "6 mar 2014"
+Date "8 mar 2014"
 Rev ""
 Comp ""
@@
 $EndComp
 $Comp
-L FE_V- #PWR51
+L FE_V- #PWR52
 U 1 1 5312A372
 P 6250 3250
-F 0 "#PWR51" H 6250 3450 40  0001 C CNN
+F 0 "#PWR52" H 6250 3450 40  0001 C CNN
 F 1 "FE_V-" H 6250 3400 40  0000 C CNN
 F 2 "" H 6250 3250 60  0000 C CNN
@@
 $EndComp
 $Comp
-L GND_FAN #PWR044
-U 1 1 53183257
+L AGND #PWR044
+U 1 1 53198B9B
+P 8350 800
+F 0 "#PWR044" H 8350 800 40  0001 C CNN
+F 1 "AGND" H 8350 730 50  0000 C CNN
+F 2 "" H 8350 800 60  0000 C CNN
+F 3 "" H 8350 800 60  0000 C CNN
+	1    8350 800
+	1    0    0    -1
+$EndComp
+$Comp
+L AGND #PWR045
+U 1 1 53198BAA
 P 7650 4400
-F 0 "#PWR044" H 7650 4400 30  0001 C CNN
-F 1 "GND_FAN" H 7650 4330 30  0000 C CNN
+F 0 "#PWR045" H 7650 4400 40  0001 C CNN
+F 1 "AGND" H 7650 4330 50  0000 C CNN
 F 2 "" H 7650 4400 60  0000 C CNN
 F 3 "" H 7650 4400 60  0000 C CNN
@@
 $EndComp
 $Comp
-L GND_FAN #PWR045
-U 1 1 53183270
-P 8350 800
-F 0 "#PWR045" H 8350 800 30  0001 C CNN
-F 1 "GND_FAN" H 8350 730 30  0000 C CNN
-F 2 "" H 8350 800 60  0000 C CNN
-F 3 "" H 8350 800 60  0000 C CNN
-	1    8350 800
-	1    0    0    -1
-$EndComp
-$Comp
-L GND_FAN #PWR046
-U 1 1 5318327F
+L AGND #PWR046
+U 1 1 53198BB9
 P 5050 3350
-F 0 "#PWR046" H 5050 3350 30  0001 C CNN
-F 1 "GND_FAN" H 5050 3280 30  0000 C CNN
+F 0 "#PWR046" H 5050 3350 40  0001 C CNN
+F 1 "AGND" H 5050 3280 50  0000 C CNN
 F 2 "" H 5050 3350 60  0000 C CNN
 F 3 "" H 5050 3350 60  0000 C CNN
@@
 $EndComp
 $Comp
-L GND_FAN #PWR047
-U 1 1 5318328E
+L AGND #PWR047
+U 1 1 53198BC8
 P 3000 3600
-F 0 "#PWR047" H 3000 3600 30  0001 C CNN
-F 1 "GND_FAN" H 3000 3530 30  0000 C CNN
+F 0 "#PWR047" H 3000 3600 40  0001 C CNN
+F 1 "AGND" H 3000 3530 50  0000 C CNN
 F 2 "" H 3000 3600 60  0000 C CNN
 F 3 "" H 3000 3600 60  0000 C CNN
@@
 $EndComp
 $Comp
-L GND_FAN #PWR048
-U 1 1 5318329D
+L AGND #PWR048
+U 1 1 53198BD7
 P 2400 1850
-F 0 "#PWR048" H 2400 1850 30  0001 C CNN
-F 1 "GND_FAN" H 2400 1780 30  0000 C CNN
+F 0 "#PWR048" H 2400 1850 40  0001 C CNN
+F 1 "AGND" H 2400 1780 50  0000 C CNN
 F 2 "" H 2400 1850 60  0000 C CNN
 F 3 "" H 2400 1850 60  0000 C CNN
