File: Power.sch (KiCad schematic (older format))
At the start: 13 parts, among them P1 24 Pin MiniFit JR, SW1 SWITCH_INV

Commit message: Power Filter Module
Created and associated footprints for PCB layout
Parts:
- L1, L2, L3: MFG NAME (none) -> Bourns Inc.; MFG PART NUM (none) -> CM322522-220KL
- SW1: value SWITCH_INV -> SWITCH; MFG NAME (none) -> C&K Components; MFG PART NUM (none) -> OS102011MA1QN1
- TH1, TH2, TH3, TH4: MFG NAME (none) -> TE Connectivity; MFG PART NUM (none) -> MINISMDC050F-2
Changed lines of the file:
@@
 Sheet 4 9
 Title ""
-Date "24 feb 2014"
+Date "25 feb 2014"
 Rev ""
 Comp ""
@@
 P 5750 3150
 F 0 "SW1" H 5550 3300 50  0000 C CNN
-F 1 "SWITCH_INV" H 5600 3000 50  0000 C CNN
+F 1 "SWITCH" H 5600 3000 50  0000 C CNN
 F 2 "~" H 5750 3150 60  0000 C CNN
 F 3 "~" H 5750 3150 60  0000 C CNN
+F 4 "C&K Components" H 5750 3150 60  0001 C CNN "MFG NAME"
+F 5 "OS102011MA1QN1" H 5750 3150 60  0001 C CNN "MFG PART NUM"
 	1    5750 3150
 	1    0    0    -1
@@
 	7200 3050 7200 2850
 $Comp
-L INDUCTOR L2
-U 1 1 52F769B8
-P 8900 3000
-F 0 "L2" V 8850 3000 40  0000 C CNN
-F 1 "INDUCTOR" V 9000 3000 40  0000 C CNN
-F 2 "~" H 8900 3000 60  0000 C CNN
-F 3 "~" H 8900 3000 60  0000 C CNN
-	1    8900 3000
-	0    -1   -1   0
-$EndComp
-$Comp
 L C C2
 U 1 1 52F769CC
@@
 	1    9350 3250
 	1    0    0    -1
-$EndComp
-$Comp
-L INDUCTOR L3
-U 1 1 52F769D9
-P 8900 4200
-F 0 "L3" V 8850 4200 40  0000 C CNN
-F 1 "INDUCTOR" V 9000 4200 40  0000 C CNN
-F 2 "~" H 8900 4200 60  0000 C CNN
-F 3 "~" H 8900 4200 60  0000 C CNN
-	1    8900 4200
-	0    -1   -1   0
 $EndComp
 $Comp
@@
 F 2 "~" H 4650 1850 60  0000 C CNN
 F 3 "~" H 4650 1850 60  0000 C CNN
+F 4 "TE Connectivity" H 4650 1850 60  0001 C CNN "MFG NAME"
+F 5 "MINISMDC050F-2" H 4650 1850 60  0001 C CNN "MFG PART NUM"
 	1    4650 1850
-	0    -1   -1   0
-$EndComp
-$Comp
-L THERMISTOR TH2
-U 1 1 52F9DF41
-P 5050 2050
-F 0 "TH2" V 5150 2100 50  0000 C CNN
-F 1 "THERMISTOR" V 4950 2050 50  0000 C CNN
-F 2 "~" H 5050 2050 60  0000 C CNN
-F 3 "~" H 5050 2050 60  0000 C CNN
-	1    5050 2050
-	0    -1   -1   0
-$EndComp
-$Comp
-L THERMISTOR TH3
-U 1 1 52F9DF47
-P 5850 2250
-F 0 "TH3" V 5950 2300 50  0000 C CNN
-F 1 "THERMISTOR" V 5750 2250 50  0000 C CNN
-F 2 "~" H 5850 2250 60  0000 C CNN
-F 3 "~" H 5850 2250 60  0000 C CNN
-	1    5850 2250
-	0    -1   -1   0
-$EndComp
-$Comp
-L THERMISTOR TH4
-U 1 1 52F9DF57
-P 6750 2450
-F 0 "TH4" V 6850 2500 50  0000 C CNN
-F 1 "THERMISTOR" V 6650 2450 50  0000 C CNN
-F 2 "~" H 6750 2450 60  0000 C CNN
-F 3 "~" H 6750 2450 60  0000 C CNN
-	1    6750 2450
 	0    -1   -1   0
 $EndComp
@@
 F 2 "~" H 8900 2150 60  0000 C CNN
 F 3 "~" H 8900 2150 60  0000 C CNN
+F 4 "Bourns Inc." H 8900 2150 60  0001 C CNN "MFG NAME"
+F 5 "CM322522-220KL" H 8900 2150 60  0001 C CNN "MFG PART NUM"
 	1    8900 2150
 	0    -1   -1   0
@@
 	1    0    0    -1
 $EndComp
+$Comp
+L THERMISTOR TH2
+U 1 1 530C510B
+P 5050 2050
+F 0 "TH2" V 5150 2100 50  0000 C CNN
+F 1 "THERMISTOR" V 4950 2050 50  0000 C CNN
+F 2 "~" H 5050 2050 60  0000 C CNN
+F 3 "~" H 5050 2050 60  0000 C CNN
+F 4 "TE Connectivity" H 5050 2050 60  0001 C CNN "MFG NAME"
+F 5 "MINISMDC050F-2" H 5050 2050 60  0001 C CNN "MFG PART NUM"
+	1    5050 2050
+	0    -1   -1   0
+$EndComp
+$Comp
+L THERMISTOR TH3
+U 1 1 530C5113
+P 5850 2250
+F 0 "TH3" V 5950 2300 50  0000 C CNN
+F 1 "THERMISTOR" V 5750 2250 50  0000 C CNN
+F 2 "~" H 5850 2250 60  0000 C CNN
+F 3 "~" H 5850 2250 60  0000 C CNN
+F 4 "TE Connectivity" H 5850 2250 60  0001 C CNN "MFG NAME"
+F 5 "MINISMDC050F-2" H 5850 2250 60  0001 C CNN "MFG PART NUM"
+	1    5850 2250
+	0    -1   -1   0
+$EndComp
+$Comp
+L THERMISTOR TH4
+U 1 1 530C511B
+P 6750 2450
+F 0 "TH4" V 6850 2500 50  0000 C CNN
+F 1 "THERMISTOR" V 6650 2450 50  0000 C CNN
+F 2 "~" H 6750 2450 60  0000 C CNN
+F 3 "~" H 6750 2450 60  0000 C CNN
+F 4 "TE Connectivity" H 6750 2450 60  0001 C CNN "MFG NAME"
+F 5 "MINISMDC050F-2" H 6750 2450 60  0001 C CNN "MFG PART NUM"
+	1    6750 2450
+	0    -1   -1   0
+$EndComp
+$Comp
+L INDUCTOR L2
+U 1 1 530C517F
+P 8900 3000
+F 0 "L2" V 8850 3000 40  0000 C CNN
+F 1 "INDUCTOR" V 9000 3000 40  0000 C CNN
+F 2 "~" H 8900 3000 60  0000 C CNN
+F 3 "~" H 8900 3000 60  0000 C CNN
+F 4 "Bourns Inc." H 8900 3000 60  0001 C CNN "MFG NAME"
+F 5 "CM322522-220KL" H 8900 3000 60  0001 C CNN "MFG PART NUM"
+	1    8900 3000
+	0    -1   -1   0
+$EndComp
+$Comp
+L INDUCTOR L3
+U 1 1 530C5187
+P 8900 4200
+F 0 "L3" V 8850 4200 40  0000 C CNN
+F 1 "INDUCTOR" V 9000 4200 40  0000 C CNN
+F 2 "~" H 8900 4200 60  0000 C CNN
+F 3 "~" H 8900 4200 60  0000 C CNN
+F 4 "Bourns Inc." H 8900 4200 60  0001 C CNN "MFG NAME"
+F 5 "CM322522-220KL" H 8900 4200 60  0001 C CNN "MFG PART NUM"
+	1    8900 4200
+	0    -1   -1   0
+$EndComp
 $EndSCHEMATC

Commit message: Layout v1.0
Connections:
- net labels removed: +3.3VP
Changed lines of the file:
@@
 Sheet 4 9
 Title ""
-Date "28 feb 2014"
+Date "3 mar 2014"
 Rev ""
 Comp ""
@@
 $EndComp
 $Comp
-L GND #PWR026
+L GND #PWR023
 U 1 1 52F7672F
 P 2650 2050
-F 0 "#PWR026" H 2650 2050 30  0001 C CNN
+F 0 "#PWR023" H 2650 2050 30  0001 C CNN
 F 1 "GND" H 2650 1980 30  0001 C CNN
 F 2 "" H 2650 2050 60  0000 C CNN
@@
 $EndComp
 $Comp
-L +5V #PWR027
+L +5V #PWR024
 U 1 1 52F7677F
 P 10150 1900
-F 0 "#PWR027" H 10150 1990 20  0001 C CNN
+F 0 "#PWR024" H 10150 1990 20  0001 C CNN
 F 1 "+5V" H 10150 1990 30  0000 C CNN
 F 2 "" H 10150 1900 60  0000 C CNN
@@
 	7150 2450 7150 1550
 $Comp
-L -12P #PWR028
+L -12P #PWR025
 U 1 1 52F768E3
 P 7150 1550
-F 0 "#PWR028" H 7150 1680 20  0001 C CNN
+F 0 "#PWR025" H 7150 1680 20  0001 C CNN
 F 1 "-12P" H 7150 1650 30  0000 C CNN
 F 2 "" H 7150 1550 60  0000 C CNN
@@
 $EndComp
 $Comp
-L +12P #PWR029
+L +12P #PWR026
 U 1 1 52F768F2
 P 6250 1550
-F 0 "#PWR029" H 6250 1520 30  0001 C CNN
+F 0 "#PWR026" H 6250 1520 30  0001 C CNN
 F 1 "+12P" H 6250 1650 30  0000 C CNN
 F 2 "" H 6250 1550 60  0000 C CNN
@@
 	5050 3150 5250 3150
 $Comp
-L GND #PWR030
+L GND #PWR027
 U 1 1 52F7693B
 P 6400 3550
-F 0 "#PWR030" H 6400 3550 30  0001 C CNN
+F 0 "#PWR027" H 6400 3550 30  0001 C CNN
 F 1 "GND" H 6400 3480 30  0001 C CNN
 F 2 "" H 6400 3550 60  0000 C CNN
@@
 	6500 3050 6250 3050
 $Comp
-L +3.3V #PWR031
+L +3.3V #PWR028
 U 1 1 52F76991
 P 7200 2850
-F 0 "#PWR031" H 7200 2810 30  0001 C CNN
+F 0 "#PWR028" H 7200 2810 30  0001 C CNN
 F 1 "+3.3V" H 7200 2960 30  0000 C CNN
 F 2 "" H 7200 2850 60  0000 C CNN
@@
 $EndComp
 $Comp
-L +12P #PWR032
+L +12P #PWR029
 U 1 1 52F769E7
 P 8100 2750
-F 0 "#PWR032" H 8100 2720 30  0001 C CNN
+F 0 "#PWR029" H 8100 2720 30  0001 C CNN
 F 1 "+12P" H 8100 2850 30  0000 C CNN
 F 2 "" H 8100 2750 60  0000 C CNN
@@
 $EndComp
 $Comp
-L GND #PWR033
+L GND #PWR030
 U 1 1 52F769F6
 P 8900 3650
-F 0 "#PWR033" H 8900 3650 30  0001 C CNN
+F 0 "#PWR030" H 8900 3650 30  0001 C CNN
 F 1 "GND" H 8900 3580 30  0001 C CNN
 F 2 "" H 8900 3650 60  0000 C CNN
@@
 $EndComp
 $Comp
-L -12P #PWR034
+L -12P #PWR031
 U 1 1 52F76A05
 P 8150 4450
-F 0 "#PWR034" H 8150 4580 20  0001 C CNN
+F 0 "#PWR031" H 8150 4580 20  0001 C CNN
 F 1 "-12P" H 8150 4550 30  0000 C CNN
 F 2 "" H 8150 4450 60  0000 C CNN
@@
 	8150 4200 8150 4450
 $Comp
-L -12V #PWR035
+L -12V #PWR032
 U 1 1 52F76AF7
 P 10200 4450
-F 0 "#PWR035" H 10200 4580 20  0001 C CNN
+F 0 "#PWR032" H 10200 4580 20  0001 C CNN
 F 1 "-12V" H 10200 4550 30  0000 C CNN
 F 2 "" H 10200 4450 60  0000 C CNN
@@
 $EndComp
 $Comp
-L +12V #PWR036
+L +12V #PWR033
 U 1 1 52F76B06
 P 10150 2750
-F 0 "#PWR036" H 10150 2700 20  0001 C CNN
+F 0 "#PWR033" H 10150 2700 20  0001 C CNN
 F 1 "+12V" H 10150 2850 30  0000 C CNN
 F 2 "" H 10150 2750 60  0000 C CNN
@@
 Connection ~ 4350 2250
 $Comp
-L +12C #PWR037
+L +12C #PWR034
 U 1 1 52F9D553
 P 4350 1600
-F 0 "#PWR037" H 4350 1570 30  0001 C CNN
+F 0 "#PWR034" H 4350 1570 30  0001 C CNN
 F 1 "+12C" H 4350 1710 40  0000 C CNN
 F 2 "" H 4350 1600 60  0000 C CNN
@@
 Connection ~ 9350 2150
 $Comp
-L GND #PWR038
+L GND #PWR035
 U 1 1 5302E727
 P 9350 2750
-F 0 "#PWR038" H 9350 2750 30  0001 C CNN
+F 0 "#PWR035" H 9350 2750 30  0001 C CNN
 F 1 "GND" H 9350 2680 30  0001 C CNN
 F 2 "" H 9350 2750 60  0000 C CNN
@@
 F 3 "" H 5450 1550 60  0000 C CNN
 	1    5450 1550
-	1    0    0    -1
-$EndComp
-$Comp
-L +3.3VP #PWR039
-U 1 1 5302E797
-P 5150 1550
-F 0 "#PWR039" H 5200 1580 20  0001 C CNN
-F 1 "+3.3VP" H 5150 1640 30  0000 C CNN
-F 2 "" H 5150 1550 60  0000 C CNN
-F 3 "" H 5150 1550 60  0000 C CNN
-	1    5150 1550
 	1    0    0    -1
 $EndComp
@@
 	0    -1   -1   0
 $EndComp
+$Comp
+L +3.3V #PWR036
+U 1 1 5312AD2B
+P 5150 1550
+F 0 "#PWR036" H 5150 1510 30  0001 C CNN
+F 1 "+3.3V" H 5150 1660 30  0000 C CNN
+F 2 "" H 5150 1550 60  0000 C CNN
+F 3 "" H 5150 1550 60  0000 C CNN
+	1    5150 1550
+	1    0    0    -1
+$EndComp
 $EndSCHEMATC

Commit message: Layout v5.0
Parts:
- added TP1: CONN_1, symbol CONN_1
Connections:
- net GND: now also TP1.1
Changed lines of the file:
@@
 Sheet 4 9
 Title ""
-Date "6 mar 2014"
+Date "8 mar 2014"
 Rev ""
 Comp ""
@@
 	9350 2600 9350 2750
 $Comp
-L +5P #PWR34
+L +5P #PWR35
 U 1 1 5302E779
 P 8100 1900
-F 0 "#PWR34" H 8100 2030 20  0001 C CNN
+F 0 "#PWR35" H 8100 2030 20  0001 C CNN
 F 1 "+5P" H 8100 2000 30  0000 C CNN
 F 2 "" H 8100 1900 60  0000 C CNN
@@
 	1    0    0    -1
 $EndComp
+$Comp
+L GND #PWR037
+U 1 1 531AD37F
+P 7800 4100
+F 0 "#PWR037" H 7800 4100 30  0001 C CNN
+F 1 "GND" H 7800 4030 30  0001 C CNN
+F 2 "" H 7800 4100 60  0000 C CNN
+F 3 "" H 7800 4100 60  0000 C CNN
+	1    7800 4100
+	1    0    0    -1
+$EndComp
+$Comp
+L CONN_1 TP1
+U 1 1 531AD387
+P 7500 3900
+F 0 "TP1" H 7580 3900 40  0000 L CNN
+F 1 "CONN_1" H 7500 3955 30  0001 C CNN
+F 2 "" H 7500 3900 60  0000 C CNN
+F 3 "" H 7500 3900 60  0000 C CNN
+	1    7500 3900
+	-1   0    0    1
+$EndComp
+Wire Wire Line
+	7650 3900 7800 3900
+Wire Wire Line
+	7800 3900 7800 4100
 $EndSCHEMATC

Commit message: Layout v6.0
Parts:
- added JP1, JP2, JP3, JP4: JUMPER, ~, symbol JUMPER
Connections:
- net +12C: now also P1.10 (P10); no longer P1.9 (P9)
- net GND: now also P1.5 (P5), JP1.1, JP2.1, JP3.1, JP4.1; no longer P1.6 (P6)
- net at P1.1 (P1), P1.2 (P2), TH1.1: now also P1.12 (P12)
- net at P1.13 (P13): no longer TH4.1
- net at P1.14 (P14): now also TH4.1
- net at P1.15 (P15): no longer SW1.2
- net at P1.16 (P16): now also SW1.2
- net at P1.4 (P4): now also P1.6 (P6), TH2.1; no longer P1.8 (P8)
- net at P1.7 (P7): now also P1.3 (P3)
- new net AGND: JP1.2
- new net GND_LED: JP4.2
- new net GND_PWR: JP3.2
- new net GND_RELAY: JP2.2
Other:
- moved on the sheet: TP1
Changed lines of the file:
@@
 Sheet 4 9
 Title ""
-Date "8 mar 2014"
+Date "9 mar 2014"
 Rev ""
 Comp ""
@@
 F 5 "39-30-1240" H 3550 2400 60  0001 C CNN "MFG PART NUM"
 	1    3550 2400
-	-1   0    0    -1
-$EndComp
-$Comp
-L GND #PWR023
+	1    0    0    -1
+$EndComp
+$Comp
+L GND #PWR26
 U 1 1 52F7672F
 P 2650 2050
-F 0 "#PWR023" H 2650 2050 30  0001 C CNN
+F 0 "#PWR26" H 2650 2050 30  0001 C CNN
 F 1 "GND" H 2650 1980 30  0001 C CNN
 F 2 "" H 2650 2050 60  0000 C CNN
@@
 $EndComp
 $Comp
-L +5V #PWR024
+L +5V #PWR45
 U 1 1 52F7677F
 P 10150 1900
-F 0 "#PWR024" H 10150 1990 20  0001 C CNN
+F 0 "#PWR45" H 10150 1990 20  0001 C CNN
 F 1 "+5V" H 10150 1990 30  0000 C CNN
 F 2 "" H 10150 1900 60  0000 C CNN
@@
 	7150 2450 7150 1550
 $Comp
-L -12P #PWR025
+L -12P #PWR38
 U 1 1 52F768E3
 P 7150 1550
-F 0 "#PWR025" H 7150 1680 20  0001 C CNN
+F 0 "#PWR38" H 7150 1680 20  0001 C CNN
 F 1 "-12P" H 7150 1650 30  0000 C CNN
 F 2 "" H 7150 1550 60  0000 C CNN
@@
 $EndComp
 $Comp
-L +12P #PWR026
+L +12P #PWR32
 U 1 1 52F768F2
 P 6250 1550
-F 0 "#PWR026" H 6250 1520 30  0001 C CNN
+F 0 "#PWR32" H 6250 1520 30  0001 C CNN
 F 1 "+12P" H 6250 1650 30  0000 C CNN
 F 2 "" H 6250 1550 60  0000 C CNN
@@
 	5050 3150 5250 3150
 $Comp
-L GND #PWR027
+L GND #PWR37
 U 1 1 52F7693B
 P 6400 3550
-F 0 "#PWR027" H 6400 3550 30  0001 C CNN
+F 0 "#PWR37" H 6400 3550 30  0001 C CNN
 F 1 "GND" H 6400 3480 30  0001 C CNN
 F 2 "" H 6400 3550 60  0000 C CNN
@@
 	6500 3050 6250 3050
 $Comp
-L +3.3V #PWR028
+L +3.3V #PWR39
 U 1 1 52F76991
 P 7200 2850
-F 0 "#PWR028" H 7200 2810 30  0001 C CNN
+F 0 "#PWR39" H 7200 2810 30  0001 C CNN
 F 1 "+3.3V" H 7200 2960 30  0000 C CNN
 F 2 "" H 7200 2850 60  0000 C CNN
@@
 $EndComp
 $Comp
-L +12P #PWR029
+L +12P #PWR41
 U 1 1 52F769E7
 P 8100 2750
-F 0 "#PWR029" H 8100 2720 30  0001 C CNN
+F 0 "#PWR41" H 8100 2720 30  0001 C CNN
 F 1 "+12P" H 8100 2850 30  0000 C CNN
 F 2 "" H 8100 2750 60  0000 C CNN
@@
 $EndComp
 $Comp
-L GND #PWR030
+L GND #PWR43
 U 1 1 52F769F6
 P 8900 3650
-F 0 "#PWR030" H 8900 3650 30  0001 C CNN
+F 0 "#PWR43" H 8900 3650 30  0001 C CNN
 F 1 "GND" H 8900 3580 30  0001 C CNN
 F 2 "" H 8900 3650 60  0000 C CNN
@@
 $EndComp
 $Comp
-L -12P #PWR031
+L -12P #PWR42
 U 1 1 52F76A05
 P 8150 4450
-F 0 "#PWR031" H 8150 4580 20  0001 C CNN
+F 0 "#PWR42" H 8150 4580 20  0001 C CNN
 F 1 "-12P" H 8150 4550 30  0000 C CNN
 F 2 "" H 8150 4450 60  0000 C CNN
@@
 	8150 4200 8150 4450
 $Comp
-L -12V #PWR032
+L -12V #PWR47
 U 1 1 52F76AF7
 P 10200 4450
-F 0 "#PWR032" H 10200 4580 20  0001 C CNN
+F 0 "#PWR47" H 10200 4580 20  0001 C CNN
 F 1 "-12V" H 10200 4550 30  0000 C CNN
 F 2 "" H 10200 4450 60  0000 C CNN
@@
 $EndComp
 $Comp
-L +12V #PWR033
+L +12V #PWR46
 U 1 1 52F76B06
 P 10150 2750
-F 0 "#PWR033" H 10150 2700 20  0001 C CNN
+F 0 "#PWR46" H 10150 2700 20  0001 C CNN
 F 1 "+12V" H 10150 2850 30  0000 C CNN
 F 2 "" H 10150 2750 60  0000 C CNN
@@
 Connection ~ 4350 2250
 $Comp
-L +12C #PWR034
+L +12C #PWR27
 U 1 1 52F9D553
 P 4350 1600
-F 0 "#PWR034" H 4350 1570 30  0001 C CNN
+F 0 "#PWR27" H 4350 1570 30  0001 C CNN
 F 1 "+12C" H 4350 1710 40  0000 C CNN
 F 2 "" H 4350 1600 60  0000 C CNN
@@
 Connection ~ 9350 2150
 $Comp
-L GND #PWR035
+L GND #PWR44
 U 1 1 5302E727
 P 9350 2750
-F 0 "#PWR035" H 9350 2750 30  0001 C CNN
+F 0 "#PWR44" H 9350 2750 30  0001 C CNN
 F 1 "GND" H 9350 2680 30  0001 C CNN
 F 2 "" H 9350 2750 60  0000 C CNN
@@
 	9350 2600 9350 2750
 $Comp
-L +5P #PWR35
+L +5P #PWR40
 U 1 1 5302E779
 P 8100 1900
-F 0 "#PWR35" H 8100 2030 20  0001 C CNN
+F 0 "#PWR40" H 8100 2030 20  0001 C CNN
 F 1 "+5P" H 8100 2000 30  0000 C CNN
 F 2 "" H 8100 1900 60  0000 C CNN
@@
 $EndComp
 $Comp
-L +5P #PWR29
+L +5P #PWR31
 U 1 1 5302E788
 P 5450 1550
-F 0 "#PWR29" H 5450 1680 20  0001 C CNN
+F 0 "#PWR31" H 5450 1680 20  0001 C CNN
 F 1 "+5P" H 5450 1650 30  0000 C CNN
 F 2 "" H 5450 1550 60  0000 C CNN
@@
 $EndComp
 $Comp
-L +3.3V #PWR036
+L +3.3V #PWR29
 U 1 1 5312AD2B
 P 5150 1550
-F 0 "#PWR036" H 5150 1510 30  0001 C CNN
+F 0 "#PWR29" H 5150 1510 30  0001 C CNN
 F 1 "+3.3V" H 5150 1660 30  0000 C CNN
 F 2 "" H 5150 1550 60  0000 C CNN
@@
 $EndComp
 $Comp
-L GND #PWR037
+L GND #PWR28
 U 1 1 531AD37F
-P 7800 4100
-F 0 "#PWR037" H 7800 4100 30  0001 C CNN
-F 1 "GND" H 7800 4030 30  0001 C CNN
-F 2 "" H 7800 4100 60  0000 C CNN
-F 3 "" H 7800 4100 60  0000 C CNN
-	1    7800 4100
+P 5000 5000
+F 0 "#PWR28" H 5000 5000 30  0001 C CNN
+F 1 "GND" H 5000 4930 30  0001 C CNN
+F 2 "" H 5000 5000 60  0000 C CNN
+F 3 "" H 5000 5000 60  0000 C CNN
+	1    5000 5000
 	1    0    0    -1
 $EndComp
@@
 L CONN_1 TP1
 U 1 1 531AD387
-P 7500 3900
-F 0 "TP1" H 7580 3900 40  0000 L CNN
-F 1 "CONN_1" H 7500 3955 30  0001 C CNN
-F 2 "" H 7500 3900 60  0000 C CNN
-F 3 "" H 7500 3900 60  0000 C CNN
-	1    7500 3900
+P 4700 4800
+F 0 "TP1" H 4780 4800 40  0000 L CNN
+F 1 "CONN_1" H 4700 4855 30  0001 C CNN
+F 2 "" H 4700 4800 60  0000 C CNN
+F 3 "" H 4700 4800 60  0000 C CNN
+	1    4700 4800
 	-1   0    0    1
 $EndComp
 Wire Wire Line
-	7650 3900 7800 3900
-Wire Wire Line
-	7800 3900 7800 4100
+	4850 4800 5000 4800
+Wire Wire Line
+	5000 4800 5000 5000
+Wire Wire Line
+	3950 2350 4250 2350
+Wire Wire Line
+	4250 2350 4250 1850
+Connection ~ 4250 1850
+$Comp
+L JUMPER JP1
+U 1 1 531BC10A
+P 5650 4350
+F 0 "JP1" H 5650 4500 60  0000 C CNN
+F 1 "JUMPER" H 5650 4270 40  0000 C CNN
+F 2 "~" H 5650 4350 60  0000 C CNN
+F 3 "~" H 5650 4350 60  0000 C CNN
+	1    5650 4350
+	1    0    0    -1
+$EndComp
+$Comp
+L JUMPER JP2
+U 1 1 531BC117
+P 5650 4700
+F 0 "JP2" H 5650 4850 60  0000 C CNN
+F 1 "JUMPER" H 5650 4620 40  0000 C CNN
+F 2 "~" H 5650 4700 60  0000 C CNN
+F 3 "~" H 5650 4700 60  0000 C CNN
+	1    5650 4700
+	1    0    0    -1
+$EndComp
+$Comp
+L JUMPER JP3
+U 1 1 531BC11D
+P 5650 5050
+F 0 "JP3" H 5650 5200 60  0000 C CNN
+F 1 "JUMPER" H 5650 4970 40  0000 C CNN
+F 2 "~" H 5650 5050 60  0000 C CNN
+F 3 "~" H 5650 5050 60  0000 C CNN
+	1    5650 5050
+	1    0    0    -1
+$EndComp
+$Comp
+L JUMPER JP4
+U 1 1 531BC123
+P 5650 5400
+F 0 "JP4" H 5650 5550 60  0000 C CNN
+F 1 "JUMPER" H 5650 5320 40  0000 C CNN
+F 2 "~" H 5650 5400 60  0000 C CNN
+F 3 "~" H 5650 5400 60  0000 C CNN
+	1    5650 5400
+	1    0    0    -1
+$EndComp
+$Comp
+L GND #PWR30
+U 1 1 531BC129
+P 5150 5800
+F 0 "#PWR30" H 5150 5800 30  0001 C CNN
+F 1 "GND" H 5150 5730 30  0001 C CNN
+F 2 "" H 5150 5800 60  0000 C CNN
+F 3 "" H 5150 5800 60  0000 C CNN
+	1    5150 5800
+	1    0    0    -1
+$EndComp
+Wire Wire Line
+	5350 4350 5150 4350
+Wire Wire Line
+	5150 4350 5150 5800
+Wire Wire Line
+	5350 4700 5150 4700
+Connection ~ 5150 4700
+Wire Wire Line
+	5350 5050 5150 5050
+Connection ~ 5150 5050
+Wire Wire Line
+	5350 5400 5150 5400
+Connection ~ 5150 5400
+$Comp
+L GND_LED #PWR36
+U 1 1 531BC258
+P 6250 5600
+F 0 "#PWR36" H 6250 5600 30  0001 C CNN
+F 1 "GND_LED" H 6250 5530 30  0000 C CNN
+F 2 "~" H 6250 5600 60  0000 C CNN
+F 3 "~" H 6250 5600 60  0000 C CNN
+	1    6250 5600
+	1    0    0    -1
+$EndComp
+$Comp
+L GND_PWR #PWR35
+U 1 1 531BC276
+P 6250 5200
+F 0 "#PWR35" H 6250 5200 30  0001 C CNN
+F 1 "GND_PWR" H 6250 5130 30  0000 C CNN
+F 2 "~" H 6250 5200 60  0000 C CNN
+F 3 "~" H 6250 5200 60  0000 C CNN
+	1    6250 5200
+	1    0    0    -1
+$EndComp
+$Comp
+L GND_RELAY #PWR34
+U 1 1 531BC285
+P 6250 4850
+F 0 "#PWR34" H 6250 4850 30  0001 C CNN
+F 1 "GND_RELAY" H 6250 4780 30  0000 C CNN
+F 2 "~" H 6250 4850 60  0000 C CNN
+F 3 "~" H 6250 4850 60  0000 C CNN
+	1    6250 4850
+	1    0    0    -1
+$EndComp
+$Comp
+L AGND #PWR33
+U 1 1 531BC294
+P 6250 4500
+F 0 "#PWR33" H 6250 4500 40  0001 C CNN
+F 1 "AGND" H 6250 4430 50  0000 C CNN
+F 2 "" H 6250 4500 60  0000 C CNN
+F 3 "" H 6250 4500 60  0000 C CNN
+	1    6250 4500
+	1    0    0    -1
+$EndComp
+Wire Wire Line
+	6250 4500 6250 4350
+Wire Wire Line
+	6250 4350 5950 4350
+Wire Wire Line
+	6250 4850 6250 4700
+Wire Wire Line
+	6250 4700 5950 4700
+Wire Wire Line
+	6250 5200 6250 5050
+Wire Wire Line
+	6250 5050 5950 5050
+Wire Wire Line
+	6250 5600 6250 5400
+Wire Wire Line
+	6250 5400 5950 5400
 $EndSCHEMATC
