File: Power.sch (KiCad schematic (older format))
At the start: 18 parts, among them P1 24 Pin MiniFit JR, SW1 SWITCH

Commit message: Layout v12.0
Connections:
- net GND: now also P1.3 (P3), P1.7 (P7)
Changed lines of the file:
@@
 Sheet 4 9
 Title ""
-Date "15 mar 2014"
+Date "16 mar 2014"
 Rev ""
 Comp ""
@@
 $EndComp
 $Comp
-L GND #PWR25
+L GND #PWR022
 U 1 1 52F7672F
 P 2650 2050
-F 0 "#PWR25" H 2650 2050 30  0001 C CNN
+F 0 "#PWR022" H 2650 2050 30  0001 C CNN
 F 1 "GND" H 2650 1980 30  0001 C CNN
 F 2 "" H 2650 2050 60  0000 C CNN
@@
 $EndComp
 $Comp
-L +5V #PWR44
+L +5V #PWR023
 U 1 1 52F7677F
 P 10150 1900
-F 0 "#PWR44" H 10150 1990 20  0001 C CNN
+F 0 "#PWR023" H 10150 1990 20  0001 C CNN
 F 1 "+5V" H 10150 1990 30  0000 C CNN
 F 2 "" H 10150 1900 60  0000 C CNN
@@
 	2650 2050 3150 2050
 Wire Wire Line
-	3150 2150 2800 2150
-Wire Wire Line
-	2800 2150 2800 1950
+	2800 2150 3150 2150
 $Comp
 L SWITCH_INV SW1
@@
 	7150 2450 7150 1550
 $Comp
-L -12P #PWR37
+L -12P #PWR024
 U 1 1 52F768E3
 P 7150 1550
-F 0 "#PWR37" H 7150 1680 20  0001 C CNN
+F 0 "#PWR024" H 7150 1680 20  0001 C CNN
 F 1 "-12P" H 7150 1650 30  0000 C CNN
 F 2 "" H 7150 1550 60  0000 C CNN
@@
 $EndComp
 $Comp
-L +12P #PWR31
+L +12P #PWR025
 U 1 1 52F768F2
 P 6250 1550
-F 0 "#PWR31" H 6250 1520 30  0001 C CNN
+F 0 "#PWR025" H 6250 1520 30  0001 C CNN
 F 1 "+12P" H 6250 1650 30  0000 C CNN
 F 2 "" H 6250 1550 60  0000 C CNN
@@
 	5050 3150 5250 3150
 $Comp
-L GND #PWR36
+L GND #PWR026
 U 1 1 52F7693B
 P 6400 3550
-F 0 "#PWR36" H 6400 3550 30  0001 C CNN
+F 0 "#PWR026" H 6400 3550 30  0001 C CNN
 F 1 "GND" H 6400 3480 30  0001 C CNN
 F 2 "" H 6400 3550 60  0000 C CNN
@@
 	6500 3050 6250 3050
 $Comp
-L +3.3V #PWR38
+L +3.3V #PWR027
 U 1 1 52F76991
 P 7200 2850
-F 0 "#PWR38" H 7200 2810 30  0001 C CNN
+F 0 "#PWR027" H 7200 2810 30  0001 C CNN
 F 1 "+3.3V" H 7200 2960 30  0000 C CNN
 F 2 "" H 7200 2850 60  0000 C CNN
@@
 $EndComp
 $Comp
-L +12P #PWR40
+L +12P #PWR028
 U 1 1 52F769E7
 P 8100 2750
-F 0 "#PWR40" H 8100 2720 30  0001 C CNN
+F 0 "#PWR028" H 8100 2720 30  0001 C CNN
 F 1 "+12P" H 8100 2850 30  0000 C CNN
 F 2 "" H 8100 2750 60  0000 C CNN
@@
 $EndComp
 $Comp
-L GND #PWR42
+L GND #PWR029
 U 1 1 52F769F6
 P 8900 3650
-F 0 "#PWR42" H 8900 3650 30  0001 C CNN
+F 0 "#PWR029" H 8900 3650 30  0001 C CNN
 F 1 "GND" H 8900 3580 30  0001 C CNN
 F 2 "" H 8900 3650 60  0000 C CNN
@@
 $EndComp
 $Comp
-L -12P #PWR41
+L -12P #PWR030
 U 1 1 52F76A05
 P 8150 4450
-F 0 "#PWR41" H 8150 4580 20  0001 C CNN
+F 0 "#PWR030" H 8150 4580 20  0001 C CNN
 F 1 "-12P" H 8150 4550 30  0000 C CNN
 F 2 "" H 8150 4450 60  0000 C CNN
@@
 	8150 4200 8150 4450
 $Comp
-L -12V #PWR46
+L -12V #PWR031
 U 1 1 52F76AF7
 P 10200 4450
-F 0 "#PWR46" H 10200 4580 20  0001 C CNN
+F 0 "#PWR031" H 10200 4580 20  0001 C CNN
 F 1 "-12V" H 10200 4550 30  0000 C CNN
 F 2 "" H 10200 4450 60  0000 C CNN
@@
 $EndComp
 $Comp
-L +12V #PWR45
+L +12V #PWR032
 U 1 1 52F76B06
 P 10150 2750
-F 0 "#PWR45" H 10150 2700 20  0001 C CNN
+F 0 "#PWR032" H 10150 2700 20  0001 C CNN
 F 1 "+12V" H 10150 2850 30  0000 C CNN
 F 2 "" H 10150 2750 60  0000 C CNN
@@
 Connection ~ 4350 2250
 $Comp
-L +12C #PWR26
+L +12C #PWR033
 U 1 1 52F9D553
 P 4350 1600
-F 0 "#PWR26" H 4350 1570 30  0001 C CNN
+F 0 "#PWR033" H 4350 1570 30  0001 C CNN
 F 1 "+12C" H 4350 1710 40  0000 C CNN
 F 2 "" H 4350 1600 60  0000 C CNN
@@
 Connection ~ 9350 2150
 $Comp
-L GND #PWR43
+L GND #PWR034
 U 1 1 5302E727
 P 9350 2750
-F 0 "#PWR43" H 9350 2750 30  0001 C CNN
+F 0 "#PWR034" H 9350 2750 30  0001 C CNN
 F 1 "GND" H 9350 2680 30  0001 C CNN
 F 2 "" H 9350 2750 60  0000 C CNN
@@
 $EndComp
 $Comp
-L +3.3V #PWR28
+L +3.3V #PWR035
 U 1 1 5312AD2B
 P 5150 1550
-F 0 "#PWR28" H 5150 1510 30  0001 C CNN
+F 0 "#PWR035" H 5150 1510 30  0001 C CNN
 F 1 "+3.3V" H 5150 1660 30  0000 C CNN
 F 2 "" H 5150 1550 60  0000 C CNN
@@
 $EndComp
 $Comp
-L GND #PWR27
+L GND #PWR036
 U 1 1 531AD37F
 P 5000 5000
-F 0 "#PWR27" H 5000 5000 30  0001 C CNN
+F 0 "#PWR036" H 5000 5000 30  0001 C CNN
 F 1 "GND" H 5000 4930 30  0001 C CNN
 F 2 "" H 5000 5000 60  0000 C CNN
@@
 $EndComp
 $Comp
-L GND #PWR29
+L GND #PWR037
 U 1 1 531BC129
 P 5150 5800
-F 0 "#PWR29" H 5150 5800 30  0001 C CNN
+F 0 "#PWR037" H 5150 5800 30  0001 C CNN
 F 1 "GND" H 5150 5730 30  0001 C CNN
 F 2 "" H 5150 5800 60  0000 C CNN
@@
 Connection ~ 5150 5400
 $Comp
-L GND_LED #PWR35
+L GND_LED #PWR038
 U 1 1 531BC258
 P 6250 5600
-F 0 "#PWR35" H 6250 5600 30  0001 C CNN
+F 0 "#PWR038" H 6250 5600 30  0001 C CNN
 F 1 "GND_LED" H 6250 5530 30  0000 C CNN
 F 2 "~" H 6250 5600 60  0000 C CNN
@@
 $EndComp
 $Comp
-L GND_PWR #PWR34
+L GND_PWR #PWR039
 U 1 1 531BC276
 P 6250 5200
-F 0 "#PWR34" H 6250 5200 30  0001 C CNN
+F 0 "#PWR039" H 6250 5200 30  0001 C CNN
 F 1 "GND_PWR" H 6250 5130 30  0000 C CNN
 F 2 "~" H 6250 5200 60  0000 C CNN
@@
 $EndComp
 $Comp
-L GND_RELAY #PWR33
+L GND_RELAY #PWR040
 U 1 1 531BC285
 P 6250 4850
-F 0 "#PWR33" H 6250 4850 30  0001 C CNN
+F 0 "#PWR040" H 6250 4850 30  0001 C CNN
 F 1 "GND_RELAY" H 6250 4780 30  0000 C CNN
 F 2 "~" H 6250 4850 60  0000 C CNN
@@
 $EndComp
 $Comp
-L AGND #PWR32
+L AGND #PWR041
 U 1 1 531BC294
 P 6250 4500
-F 0 "#PWR32" H 6250 4500 40  0001 C CNN
+F 0 "#PWR041" H 6250 4500 40  0001 C CNN
 F 1 "AGND" H 6250 4430 50  0000 C CNN
 F 2 "" H 6250 4500 60  0000 C CNN
@@
 Wire Wire Line
 	6250 5400 5950 5400
+Wire Wire Line
+	2800 1950 2800 2150
+Connection ~ 2800 2050
 $EndSCHEMATC
