File: Power_Adjustment_Monitor.sch (KiCad schematic (older format))
At the start: 24 parts, among them U10 LM317K, U7 LM337T, U8 LM317K, U9 LM337T

Commit message: Layout v5.0
Connections:
- net labels added: AGND
- net labels removed: GND_TC
Changed lines of the file:
@@
 Sheet 8 9
 Title ""
-Date "6 mar 2014"
+Date "8 mar 2014"
 Rev ""
 Comp ""
@@
 $EndComp
 $Comp
-L FE_V- #PWR61
+L FE_V- #PWR62
 U 1 1 52F83296
 P 4800 5450
-F 0 "#PWR61" H 4800 5650 40  0001 C CNN
+F 0 "#PWR62" H 4800 5650 40  0001 C CNN
 F 1 "FE_V-" H 4800 5600 40  0000 C CNN
 F 2 "" H 4800 5450 60  0000 C CNN
@@
 	1    0    0    -1
 $EndComp
-$Comp
-L GND_TC #PWR059
-U 1 1 53184501
-P 4950 4300
-F 0 "#PWR059" H 4950 4300 30  0001 C CNN
-F 1 "GND_TC" H 4950 4230 30  0000 C CNN
-F 2 "" H 4950 4300 60  0000 C CNN
-F 3 "" H 4950 4300 60  0000 C CNN
-	1    4950 4300
-	1    0    0    -1
-$EndComp
 Connection ~ 2750 6100
 Connection ~ 4750 2250
@@
 Connection ~ 3050 800
 Connection ~ 2750 4150
+$Comp
+L AGND #PWR059
+U 1 1 53199459
+P 4950 4300
+F 0 "#PWR059" H 4950 4300 40  0001 C CNN
+F 1 "AGND" H 4950 4230 50  0000 C CNN
+F 2 "" H 4950 4300 60  0000 C CNN
+F 3 "" H 4950 4300 60  0000 C CNN
+	1    4950 4300
+	1    0    0    -1
+$EndComp
 $EndSCHEMATC

Commit message: Layout v16.0
Parts:
- removed U10, U8: LM317K, TO-220, symbol LM317K
- added TP10: FE_V-, symbol CONN_1
- added TP11: AGND, symbol CONN_1
- added TP8: GND_PWR, symbol CONN_1
- added TP9: FE_V+, symbol CONN_1
- added U10, U8: LM317T, TO-220, symbol LM317T
Connections:
- net +12V: now also U10.3 (IN), U8.3 (IN)
- net AGND: now also TP11.1
- net FE_V+: now also TP9.1, U10.2 (OUT)
- net FE_V-: now also TP10.1
- net GND_PWR: now also TP8.1
- net V+_ADJ: now also U8.2 (OUT)
- net at R34.2, R35.1: now also U8.1 (ADJ)
- net at R50.2, R51.1: now also U10.1 (ADJ)
Changed lines of the file:
@@
 Sheet 8 9
 Title ""
-Date "17 mar 2014"
+Date "22 mar 2014"
 Rev ""
 Comp ""
@@
 Wire Wire Line
 	3050 1500 3050 2250
-$Comp
-L LM317K U10
-U 1 1 53143282
-P 3600 850
-F 0 "U10" H 3400 1050 40  0000 C CNN
-F 1 "LM317K" H 3600 1050 40  0000 L CNN
-F 2 "TO-220" H 3600 950 30  0000 C CIN
-F 3 "~" H 3600 850 60  0000 C CNN
-	1    3600 850
-	1    0    0    -1
-$EndComp
-$Comp
-L LM317K U8
-U 1 1 531432A3
-P 3600 2750
-F 0 "U8" H 3400 2950 40  0000 C CNN
-F 1 "LM317K" H 3600 2950 40  0000 L CNN
-F 2 "TO-220" H 3600 2850 30  0000 C CIN
-F 3 "~" H 3600 2750 60  0000 C CNN
-	1    3600 2750
-	1    0    0    -1
-$EndComp
 Wire Wire Line
 	2750 4150 4950 4150
@@
 	2750 3750 2750 4550
 Wire Wire Line
-	4950 4150 4950 4300
+	4950 3950 4950 4300
 Wire Wire Line
 	4950 1700 4950 2250
@@
 	1    0    0    -1
 $EndComp
+$Comp
+L LM317T U8
+U 1 1 532BDBB1
+P 3600 850
+F 0 "U8" H 3400 1050 40  0000 C CNN
+F 1 "LM317T" H 3600 1050 40  0000 L CNN
+F 2 "TO-220" H 3600 950 30  0000 C CIN
+F 3 "~" H 3600 850 60  0000 C CNN
+	1    3600 850
+	1    0    0    -1
+$EndComp
+$Comp
+L LM317T U10
+U 1 1 532BDBBE
+P 3600 2750
+F 0 "U10" H 3400 2950 40  0000 C CNN
+F 1 "LM317T" H 3600 2950 40  0000 L CNN
+F 2 "TO-220" H 3600 2850 30  0000 C CIN
+F 3 "~" H 3600 2750 60  0000 C CNN
+	1    3600 2750
+	1    0    0    -1
+$EndComp
+$Comp
+L CONN_1 TP8
+U 1 1 532D5229
+P 4050 1950
+F 0 "TP8" H 4130 1950 40  0000 L CNN
+F 1 "GND_PWR" H 4050 2005 30  0001 C CNN
+F 2 "" H 4050 1950 60  0000 C CNN
+F 3 "" H 4050 1950 60  0000 C CNN
+	1    4050 1950
+	0    -1   -1   0
+$EndComp
+Wire Wire Line
+	4050 2100 4050 2250
+Connection ~ 4050 2250
+$Comp
+L CONN_1 TP9
+U 1 1 532D528D
+P 4600 2450
+F 0 "TP9" H 4680 2450 40  0000 L CNN
+F 1 "FE_V+" H 4600 2505 30  0001 C CNN
+F 2 "" H 4600 2450 60  0000 C CNN
+F 3 "" H 4600 2450 60  0000 C CNN
+	1    4600 2450
+	0    -1   -1   0
+$EndComp
+Wire Wire Line
+	4600 2600 4600 2700
+Connection ~ 4600 2700
+$Comp
+L CONN_1 TP10
+U 1 1 532D52F2
+P 4750 5150
+F 0 "TP10" H 4830 5150 40  0000 L CNN
+F 1 "FE_V-" H 4750 5205 30  0001 C CNN
+F 2 "" H 4750 5150 60  0000 C CNN
+F 3 "" H 4750 5150 60  0000 C CNN
+	1    4750 5150
+	0    1    -1   0
+$EndComp
+Wire Wire Line
+	4750 5300 4750 5450
+Connection ~ 4750 5450
+$Comp
+L CONN_1 TP11
+U 1 1 532D5368
+P 4950 3800
+F 0 "TP11" H 5030 3800 40  0000 L CNN
+F 1 "AGND" H 4950 3855 30  0001 C CNN
+F 2 "" H 4950 3800 60  0000 C CNN
+F 3 "" H 4950 3800 60  0000 C CNN
+	1    4950 3800
+	0    -1   -1   0
+$EndComp
+Connection ~ 4950 4150
 $EndSCHEMATC
