File: Power_Adjustment_Monitor.sch (KiCad schematic (older format))
At the start: 28 parts, among them U10 LM317T, U7 LM337T, U8 LM317T, U9 LM337T

Commit message: Layout v17.0
Other:
- moved on the sheet: TP9
