File: Arduino.sch (KiCad schematic (older format))
At the start: 21 parts

Commit message: Layout v11.0
Connections:
- net MISO: now also R15.2; no longer R14.2
- net MOSI: now also R14.2; no longer R15.2
Changed lines of the file:
@@
 Sheet 2 9
 Title ""
-Date "10 mar 2014"
+Date "15 mar 2014"
 Rev ""
 Comp ""
@@
 Text HLabel 7000 4150 2    60   Output ~ 0
 RELAY-
-Text HLabel 7000 1850 2    60   Output ~ 0
+Text HLabel 7000 1650 2    60   Output ~ 0
 MOSI
-Text HLabel 7000 1650 2    60   Input ~ 0
+Text HLabel 7000 1850 2    60   Input ~ 0
 MISO
 Text HLabel 7000 1450 2    60   Output ~ 0

Commit message: Layout v12.0
Connections:
- net at R20.1: now also ARD1.17 (DIGITAL6); no longer ARD1.12 (DIGITAL1)
Other:
- moved on the sheet: R19, R20, R42, R43, R46, R47
