File: Relay.sch (KiCad schematic (older format))
At the start: 11 parts, among them K1 RELAY, Q1 2N3904, U1 OPTO_TRANSISTOR

Commit message: Layout v8.0
Connections:
- net +12V renamed +12P
Changed lines of the file:
@@
 Sheet 7 9
 Title ""
-Date "9 mar 2014"
+Date "10 mar 2014"
 Rev ""
 Comp ""
@@
 	6650 5400 6650 5100
 $Comp
-L +12V #PWR62
-U 1 1 52F74537
-P 7400 2050
-F 0 "#PWR62" H 7400 2000 20  0001 C CNN
-F 1 "+12V" H 7400 2150 30  0000 C CNN
-F 2 "" H 7400 2050 60  0000 C CNN
-F 3 "" H 7400 2050 60  0000 C CNN
-	1    7400 2050
-	1    0    0    -1
-$EndComp
-$Comp
 L R R4
 U 1 1 52F74544
@@
 	1    0    0    -1
 $EndComp
+$Comp
+L +12P #PWR?
+U 1 1 531D6008
+P 7400 2050
+F 0 "#PWR?" H 7400 2020 30  0001 C CNN
+F 1 "+12P" H 7400 2150 30  0000 C CNN
+F 2 "" H 7400 2050 60  0000 C CNN
+F 3 "" H 7400 2050 60  0000 C CNN
+	1    7400 2050
+	1    0    0    -1
+$EndComp

Commit message: Layout v16.0
Parts:
- added TP6: +12P, symbol CONN_1
- added TP7: RLY-, symbol CONN_1
Connections:
- net +12P: now also TP6.1
- net at D2.1 (A), K1.5 (COIL-), Q1.3 (C): now also TP7.1
Changed lines of the file:
@@
 Sheet 7 9
 Title ""
-Date "17 mar 2014"
+Date "22 mar 2014"
 Rev ""
 Comp ""
@@
 	1    0    0    -1
 $EndComp
+$Comp
+L CONN_1 TP7
+U 1 1 532D5023
+P 8450 3400
+F 0 "TP7" H 8530 3400 40  0000 L CNN
+F 1 "RLY-" H 8450 3455 30  0001 C CNN
+F 2 "" H 8450 3400 60  0000 C CNN
+F 3 "" H 8450 3400 60  0000 C CNN
+	1    8450 3400
+	1    0    0    -1
+$EndComp
+Wire Wire Line
+	8300 3400 8200 3400
+Connection ~ 8200 3400
+$Comp
+L CONN_1 TP6
+U 1 1 532D507C
+P 7800 1950
+F 0 "TP6" H 7880 1950 40  0000 L CNN
+F 1 "+12P" H 7800 2005 30  0001 C CNN
+F 2 "" H 7800 1950 60  0000 C CNN
+F 3 "" H 7800 1950 60  0000 C CNN
+	1    7800 1950
+	0    -1   -1   0
+$EndComp
+Wire Wire Line
+	7800 2100 7800 2150
+Connection ~ 7800 2150
 $EndSCHEMATC
