File: Terminal_Block.sch (KiCad schematic (older format))
At the start: 2 parts, among them P4 12 Pin Terminal Block, P5 CONN_3

Commit message: Layout v11.0
Connections:
- net TC_IN_+: now also P4.6 (P6); no longer P4.7 (P7)
- net TC_IN_-: now also P4.7 (P7); no longer P4.6 (P6)
Changed lines of the file:
@@
 Sheet 9 9
 Title ""
-Date "10 mar 2014"
+Date "15 mar 2014"
 Rev ""
 Comp ""
@@
 RELAY_COM
 $Comp
-L +3.3V #PWR73
+L +3.3V #PWR72
 U 1 1 52F91565
 P 3900 1550
-F 0 "#PWR73" H 3900 1510 30  0001 C CNN
+F 0 "#PWR72" H 3900 1510 30  0001 C CNN
 F 1 "+3.3V" H 3900 1660 30  0000 C CNN
 F 2 "" H 3900 1550 60  0000 C CNN
@@
 $EndComp
 $Comp
-L +5V #PWR74
+L +5V #PWR73
 U 1 1 52F91574
 P 4150 1450
-F 0 "#PWR74" H 4150 1540 20  0001 C CNN
+F 0 "#PWR73" H 4150 1540 20  0001 C CNN
 F 1 "+5V" H 4150 1540 30  0000 C CNN
 F 2 "" H 4150 1450 60  0000 C CNN
@@
 Wire Wire Line
 	4150 1500 4150 1450
+Text HLabel 4750 1400 0    60   Output ~ 0
+TC_IN_-
 Text HLabel 4750 1300 0    60   Output ~ 0
-TC_IN_-
-Text HLabel 4750 1400 0    60   Output ~ 0
 TC_IN_+
 $Comp
@@
 	4750 1400 6200 1400
 $Comp
-L GND_PWR #PWR75
+L GND_PWR #PWR74
 U 1 1 53199927
 P 4750 1600
-F 0 "#PWR75" H 4750 1600 30  0001 C CNN
+F 0 "#PWR74" H 4750 1600 30  0001 C CNN
 F 1 "GND_PWR" H 4750 1530 30  0000 C CNN
 F 2 "~" H 4750 1600 60  0000 C CNN

Commit message: Layout v13.0
Parts:
- added C22, C23, C24, C25: C, SM1210, symbol C
- added R52: R, SM0805, symbol R
Connections:
- net +3.3V: now also C23.1
- net +5V: now also C22.1
- net GND_PWR: now also C22.2, C23.2, C24.2, C25.2, R52.1
- net TACH: now also R52.2
- net V+_ADJ: now also C25.1
- net V-_ADJ: now also C24.1
Other:
- moved on the sheet: P5
Changed lines of the file:
@@
 Sheet 9 9
 Title ""
-Date "16 mar 2014"
+Date "17 mar 2014"
 Rev ""
 Comp ""
@@
 Text HLabel 4750 900  0    60   Input ~ 0
 LED-
-Text HLabel 4750 2400 0    60   BiDi ~ 0
+Text HLabel 4750 3350 0    60   BiDi ~ 0
 RELAY_NC
-Text HLabel 4750 2200 0    60   BiDi ~ 0
+Text HLabel 4750 3150 0    60   BiDi ~ 0
 RELAY_NO
-Text HLabel 4750 2300 0    60   BiDi ~ 0
+Text HLabel 4750 3250 0    60   BiDi ~ 0
 RELAY_COM
 $Comp
-L +3.3V #PWR064
+L +3.3V #PWR72
 U 1 1 52F91565
 P 3900 1550
-F 0 "#PWR064" H 3900 1510 30  0001 C CNN
+F 0 "#PWR72" H 3900 1510 30  0001 C CNN
 F 1 "+3.3V" H 3900 1660 30  0000 C CNN
 F 2 "" H 3900 1550 60  0000 C CNN
@@
 $EndComp
 $Comp
-L +5V #PWR065
+L +5V #PWR73
 U 1 1 52F91574
 P 4150 1450
-F 0 "#PWR065" H 4150 1540 20  0001 C CNN
+F 0 "#PWR73" H 4150 1540 20  0001 C CNN
 F 1 "+5V" H 4150 1540 30  0000 C CNN
 F 2 "" H 4150 1450 60  0000 C CNN
@@
 L CONN_3 P5
 U 1 1 5309D123
-P 6550 2300
-F 0 "P5" V 6500 2300 50  0000 C CNN
-F 1 "CONN_3" V 6600 2300 40  0000 C CNN
-F 2 "" H 6550 2300 60  0000 C CNN
-F 3 "" H 6550 2300 60  0000 C CNN
-F 4 "PHOENIX CONTACT" H 6550 2300 60  0001 C CNN "MFG NAME"
-F 5 "1935174" H 6550 2300 60  0001 C CNN "MFG PART NUM"
-	1    6550 2300
-	1    0    0    -1
-$EndComp
-Wire Wire Line
-	4750 2200 6200 2200
-Wire Wire Line
-	4750 2300 6200 2300
-Wire Wire Line
-	4750 2400 6200 2400
+P 6550 3250
+F 0 "P5" V 6500 3250 50  0000 C CNN
+F 1 "CONN_3" V 6600 3250 40  0000 C CNN
+F 2 "" H 6550 3250 60  0000 C CNN
+F 3 "" H 6550 3250 60  0000 C CNN
+F 4 "PHOENIX CONTACT" H 6550 3250 60  0001 C CNN "MFG NAME"
+F 5 "1935174" H 6550 3250 60  0001 C CNN "MFG PART NUM"
+	1    6550 3250
+	1    0    0    -1
+$EndComp
+Wire Wire Line
+	4750 3150 6200 3150
+Wire Wire Line
+	4750 3250 6200 3250
+Wire Wire Line
+	4750 3350 6200 3350
 Wire Wire Line
 	4150 1500 6200 1500
@@
 	4750 1400 6200 1400
 $Comp
-L GND_PWR #PWR066
+L GND_PWR #PWR74
 U 1 1 53199927
 P 4750 1600
-F 0 "#PWR066" H 4750 1600 30  0001 C CNN
+F 0 "#PWR74" H 4750 1600 30  0001 C CNN
 F 1 "GND_PWR" H 4750 1530 30  0000 C CNN
 F 2 "~" H 4750 1600 60  0000 C CNN
@@
 	0    1    1    0
 $EndComp
+$Comp
+L R R52
+U 1 1 53263BF3
+P 6100 2300
+F 0 "R52" V 6180 2300 40  0000 C CNN
+F 1 "R" V 6107 2301 40  0000 C CNN
+F 2 "SM0805" V 6030 2300 30  0000 C CNN
+F 3 "~" H 6100 2300 30  0000 C CNN
+	1    6100 2300
+	1    0    0    1
+$EndComp
+$Comp
+L GND_PWR #PWR79
+U 1 1 53263C00
+P 6100 2700
+F 0 "#PWR79" H 6100 2700 30  0001 C CNN
+F 1 "GND_PWR" H 6100 2630 30  0000 C CNN
+F 2 "~" H 6100 2700 60  0000 C CNN
+F 3 "~" H 6100 2700 60  0000 C CNN
+	1    6100 2700
+	1    0    0    -1
+$EndComp
+Wire Wire Line
+	6100 2550 6100 2700
+Wire Wire Line
+	6100 2050 6100 1000
+Connection ~ 6100 1000
+$Comp
+L C C25
+U 1 1 53263C59
+P 5750 2300
+F 0 "C25" H 5750 2400 40  0000 L CNN
+F 1 "C" H 5756 2215 40  0000 L CNN
+F 2 "SM1210" H 5788 2150 30  0000 C CNN
+F 3 "~" H 5750 2300 60  0000 C CNN
+	1    5750 2300
+	1    0    0    -1
+$EndComp
+$Comp
+L GND_PWR #PWR78
+U 1 1 53263C78
+P 5750 2700
+F 0 "#PWR78" H 5750 2700 30  0001 C CNN
+F 1 "GND_PWR" H 5750 2630 30  0000 C CNN
+F 2 "~" H 5750 2700 60  0000 C CNN
+F 3 "~" H 5750 2700 60  0000 C CNN
+	1    5750 2700
+	1    0    0    -1
+$EndComp
+Wire Wire Line
+	5750 2500 5750 2700
+$Comp
+L GND_PWR #PWR77
+U 1 1 53263C80
+P 5500 2700
+F 0 "#PWR77" H 5500 2700 30  0001 C CNN
+F 1 "GND_PWR" H 5500 2630 30  0000 C CNN
+F 2 "~" H 5500 2700 60  0000 C CNN
+F 3 "~" H 5500 2700 60  0000 C CNN
+	1    5500 2700
+	1    0    0    -1
+$EndComp
+Wire Wire Line
+	5500 2500 5500 2700
+$Comp
+L GND_PWR #PWR76
+U 1 1 53263C87
+P 5250 2700
+F 0 "#PWR76" H 5250 2700 30  0001 C CNN
+F 1 "GND_PWR" H 5250 2630 30  0000 C CNN
+F 2 "~" H 5250 2700 60  0000 C CNN
+F 3 "~" H 5250 2700 60  0000 C CNN
+	1    5250 2700
+	1    0    0    -1
+$EndComp
+Wire Wire Line
+	5250 2500 5250 2700
+$Comp
+L GND_PWR #PWR75
+U 1 1 53263C95
+P 5000 2700
+F 0 "#PWR75" H 5000 2700 30  0001 C CNN
+F 1 "GND_PWR" H 5000 2630 30  0000 C CNN
+F 2 "~" H 5000 2700 60  0000 C CNN
+F 3 "~" H 5000 2700 60  0000 C CNN
+	1    5000 2700
+	1    0    0    -1
+$EndComp
+Wire Wire Line
+	5000 2500 5000 2700
+Wire Wire Line
+	5750 2100 5750 1900
+Connection ~ 5750 1900
+Wire Wire Line
+	5500 2100 5500 1800
+Connection ~ 5500 1800
+Wire Wire Line
+	5250 2100 5250 1700
+Connection ~ 5250 1700
+Wire Wire Line
+	5000 2100 5000 1500
+Connection ~ 5000 1500
+$Comp
+L C C24
+U 1 1 53264354
+P 5500 2300
+F 0 "C24" H 5500 2400 40  0000 L CNN
+F 1 "C" H 5506 2215 40  0000 L CNN
+F 2 "SM1210" H 5538 2150 30  0000 C CNN
+F 3 "~" H 5500 2300 60  0000 C CNN
+	1    5500 2300
+	1    0    0    -1
+$EndComp
+$Comp
+L C C23
+U 1 1 5326435A
+P 5250 2300
+F 0 "C23" H 5250 2400 40  0000 L CNN
+F 1 "C" H 5256 2215 40  0000 L CNN
+F 2 "SM1210" H 5288 2150 30  0000 C CNN
+F 3 "~" H 5250 2300 60  0000 C CNN
+	1    5250 2300
+	1    0    0    -1
+$EndComp
+$Comp
+L C C22
+U 1 1 53264360
+P 5000 2300
+F 0 "C22" H 5000 2400 40  0000 L CNN
+F 1 "C" H 5006 2215 40  0000 L CNN
+F 2 "SM1210" H 5038 2150 30  0000 C CNN
+F 3 "~" H 5000 2300 60  0000 C CNN
+	1    5000 2300
+	1    0    0    -1
+$EndComp
 $EndSCHEMATC

Commit message: Layout v17.0
Connections:
- net TC_IN_+: now also P4.7 (P7); no longer P4.6 (P6)
- net TC_IN_-: now also P4.6 (P6); no longer P4.7 (P7)
Changed lines of the file:
@@
 Sheet 9 9
 Title ""
-Date "22 mar 2014"
+Date "23 mar 2014"
 Rev ""
 Comp ""
@@
 RELAY_COM
 $Comp
-L +3.3V #PWR064
+L +3.3V #PWR76
 U 1 1 52F91565
 P 3900 1550
-F 0 "#PWR064" H 3900 1510 30  0001 C CNN
+F 0 "#PWR76" H 3900 1510 30  0001 C CNN
 F 1 "+3.3V" H 3900 1660 30  0000 C CNN
 F 2 "" H 3900 1550 60  0000 C CNN
@@
 $EndComp
 $Comp
-L +5V #PWR065
+L +5V #PWR77
 U 1 1 52F91574
 P 4150 1450
-F 0 "#PWR065" H 4150 1540 20  0001 C CNN
+F 0 "#PWR77" H 4150 1540 20  0001 C CNN
 F 1 "+5V" H 4150 1540 30  0000 C CNN
 F 2 "" H 4150 1450 60  0000 C CNN
@@
 Wire Wire Line
 	4150 1500 4150 1450
+Text HLabel 4750 1300 0    60   Output ~ 0
+TC_IN_-
 Text HLabel 4750 1400 0    60   Output ~ 0
-TC_IN_-
-Text HLabel 4750 1300 0    60   Output ~ 0
 TC_IN_+
 $Comp
@@
 	4750 1400 6200 1400
 $Comp
-L GND_PWR #PWR066
+L GND_PWR #PWR78
 U 1 1 53199927
 P 4750 1600
-F 0 "#PWR066" H 4750 1600 30  0001 C CNN
+F 0 "#PWR78" H 4750 1600 30  0001 C CNN
 F 1 "GND_PWR" H 4750 1530 30  0000 C CNN
 F 2 "~" H 4750 1600 60  0000 C CNN
@@
 $EndComp
 $Comp
-L GND_PWR #PWR067
+L GND_PWR #PWR83
 U 1 1 53263C00
 P 6100 2700
-F 0 "#PWR067" H 6100 2700 30  0001 C CNN
+F 0 "#PWR83" H 6100 2700 30  0001 C CNN
 F 1 "GND_PWR" H 6100 2630 30  0000 C CNN
 F 2 "~" H 6100 2700 60  0000 C CNN
@@
 $EndComp
 $Comp
-L GND_PWR #PWR068
+L GND_PWR #PWR82
 U 1 1 53263C78
 P 5750 2700
-F 0 "#PWR068" H 5750 2700 30  0001 C CNN
+F 0 "#PWR82" H 5750 2700 30  0001 C CNN
 F 1 "GND_PWR" H 5750 2630 30  0000 C CNN
 F 2 "~" H 5750 2700 60  0000 C CNN
@@
 	5750 2500 5750 2700
 $Comp
-L GND_PWR #PWR069
+L GND_PWR #PWR81
 U 1 1 53263C80
 P 5500 2700
-F 0 "#PWR069" H 5500 2700 30  0001 C CNN
+F 0 "#PWR81" H 5500 2700 30  0001 C CNN
 F 1 "GND_PWR" H 5500 2630 30  0000 C CNN
 F 2 "~" H 5500 2700 60  0000 C CNN
@@
 	5500 2500 5500 2700
 $Comp
-L GND_PWR #PWR070
+L GND_PWR #PWR80
 U 1 1 53263C87
 P 5250 2700
-F 0 "#PWR070" H 5250 2700 30  0001 C CNN
+F 0 "#PWR80" H 5250 2700 30  0001 C CNN
 F 1 "GND_PWR" H 5250 2630 30  0000 C CNN
 F 2 "~" H 5250 2700 60  0000 C CNN
@@
 	5250 2500 5250 2700
 $Comp
-L GND_PWR #PWR071
+L GND_PWR #PWR79
 U 1 1 53263C95
 P 5000 2700
-F 0 "#PWR071" H 5000 2700 30  0001 C CNN
+F 0 "#PWR79" H 5000 2700 30  0001 C CNN
 F 1 "GND_PWR" H 5000 2630 30  0000 C CNN
 F 2 "~" H 5000 2700 60  0000 C CNN
