File: Thermocouple.sch (KiCad schematic (older format))
At the start: 20 parts, among them P2 CONN_2, P3 CONN_3X2, U2 MCP3901, U3 LMT84, U4 OPA4170

Commit message: Layout v11.0
Parts:
- added L5: INDUCTOR, SM0805, symbol INDUCTOR
Connections:
- net +5V: now also L5.1; no longer C6.1, U2.2 (DVDD)
- new net: C6.1, L5.2, U2.2 (DVDD)
Other:
- moved on the sheet: C6, C7
Changed lines of the file:
@@
 Sheet 3 9
 Title ""
-Date "10 mar 2014"
+Date "15 mar 2014"
 Rev ""
 Comp ""
@@
 $EndComp
 $Comp
-L -12V #PWR24
+L -12V #PWR23
 U 1 1 52F4A357
 P 10250 5500
-F 0 "#PWR24" H 10250 5630 20  0001 C CNN
+F 0 "#PWR23" H 10250 5630 20  0001 C CNN
 F 1 "-12V" H 10250 5600 30  0000 C CNN
 F 2 "" H 10250 5500 60  0000 C CNN
@@
 $EndComp
 $Comp
-L +12V #PWR22
+L +12V #PWR21
 U 1 1 52F4A37C
 P 9900 5500
-F 0 "#PWR22" H 9900 5450 20  0001 C CNN
+F 0 "#PWR21" H 9900 5450 20  0001 C CNN
 F 1 "+12V" H 9900 5600 30  0000 C CNN
 F 2 "" H 9900 5500 60  0000 C CNN
@@
 	6050 6800 6050 6650
 $Comp
-L +5V #PWR14
+L +5V #PWR13
 U 1 1 53096E41
 P 5900 5250
-F 0 "#PWR14" H 5900 5340 20  0001 C CNN
+F 0 "#PWR13" H 5900 5340 20  0001 C CNN
 F 1 "+5V" H 5900 5340 30  0000 C CNN
 F 2 "" H 5900 5250 60  0000 C CNN
@@
 	6550 5300 6550 5850
 $Comp
-L +5V #PWR8
+L +5V #PWR7
 U 1 1 53097117
-P 2950 1100
-F 0 "#PWR8" H 2950 1190 20  0001 C CNN
-F 1 "+5V" H 2950 1190 30  0000 C CNN
-F 2 "" H 2950 1100 60  0000 C CNN
-F 3 "" H 2950 1100 60  0000 C CNN
-	1    2950 1100
-	1    0    0    -1
-$EndComp
-Wire Wire Line
-	2950 1100 2950 1250
+P 2950 750
+F 0 "#PWR7" H 2950 840 20  0001 C CNN
+F 1 "+5V" H 2950 840 30  0000 C CNN
+F 2 "" H 2950 750 60  0000 C CNN
+F 3 "" H 2950 750 60  0000 C CNN
+	1    2950 750
+	1    0    0    -1
+$EndComp
 Text GLabel 4450 1800 2    60   Input ~ 0
 REF+
@@
 L C C7
 U 1 1 53097282
-P 3250 1150
-F 0 "C7" H 3250 1250 40  0000 L CNN
-F 1 "C" H 3256 1065 40  0000 L CNN
-F 2 "~" H 3288 1000 30  0000 C CNN
-F 3 "~" H 3250 1150 60  0000 C CNN
-	1    3250 1150
+P 3450 1150
+F 0 "C7" H 3450 1250 40  0000 L CNN
+F 1 "C" H 3456 1065 40  0000 L CNN
+F 2 "~" H 3488 1000 30  0000 C CNN
+F 3 "~" H 3450 1150 60  0000 C CNN
+	1    3450 1150
 	0    -1   -1   0
 $EndComp
 Wire Wire Line
-	3050 1150 2950 1150
-Connection ~ 2950 1150
-Wire Wire Line
-	3550 1250 3550 1150
-Wire Wire Line
-	3550 1150 3450 1150
-$Comp
-L +5V #PWR6
-U 1 1 5309733E
-P 2500 1100
-F 0 "#PWR6" H 2500 1190 20  0001 C CNN
-F 1 "+5V" H 2500 1190 30  0000 C CNN
-F 2 "" H 2500 1100 60  0000 C CNN
-F 3 "" H 2500 1100 60  0000 C CNN
-	1    2500 1100
-	-1   0    0    -1
-$EndComp
-Wire Wire Line
-	2500 1100 2500 1250
+	3750 1250 3750 1150
+Wire Wire Line
+	3750 1150 3650 1150
 $Comp
 L C C6
 U 1 1 53097345
-P 2200 1150
-F 0 "C6" H 2200 1250 40  0000 L CNN
-F 1 "C" H 2206 1065 40  0000 L CNN
-F 2 "~" H 2238 1000 30  0000 C CNN
-F 3 "~" H 2200 1150 60  0000 C CNN
-	1    2200 1150
+P 1800 1150
+F 0 "C6" H 1800 1250 40  0000 L CNN
+F 1 "C" H 1806 1065 40  0000 L CNN
+F 2 "~" H 1838 1000 30  0000 C CNN
+F 3 "~" H 1800 1150 60  0000 C CNN
+	1    1800 1150
 	0    1    -1   0
 $EndComp
 Wire Wire Line
-	2400 1150 2500 1150
-Connection ~ 2500 1150
-Wire Wire Line
-	1900 1150 2000 1150
-Wire Wire Line
-	1900 1150 1900 1250
+	1500 1150 1600 1150
+Wire Wire Line
+	1500 1150 1500 1250
 Wire Wire Line
 	2500 5100 2500 5250
@@
 	1300 4500 1400 4500
 $Comp
-L FE_V- #PWR16
+L FE_V- #PWR15
 U 1 1 5312A19A
 P 6050 2850
-F 0 "#PWR16" H 6050 3050 40  0001 C CNN
+F 0 "#PWR15" H 6050 3050 40  0001 C CNN
 F 1 "FE_V-" H 6050 3000 40  0000 C CNN
 F 2 "" H 6050 2850 60  0000 C CNN
@@
 $EndComp
 $Comp
-L FE_V+ #PWR17
+L FE_V+ #PWR16
 U 1 1 5312A1A0
 P 6050 3850
-F 0 "#PWR17" H 6050 3950 30  0001 C CNN
+F 0 "#PWR16" H 6050 3950 30  0001 C CNN
 F 1 "FE_V+" H 6050 3950 30  0000 C CNN
 F 2 "" H 6050 3850 60  0000 C CNN
@@
 $EndComp
 $Comp
-L FE_V- #PWR20
+L FE_V- #PWR19
 U 1 1 5312A1BA
 P 8200 4050
-F 0 "#PWR20" H 8200 4250 40  0001 C CNN
+F 0 "#PWR19" H 8200 4250 40  0001 C CNN
 F 1 "FE_V-" H 8200 4200 40  0000 C CNN
 F 2 "" H 8200 4050 60  0000 C CNN
@@
 $EndComp
 $Comp
-L FE_V+ #PWR21
+L FE_V+ #PWR20
 U 1 1 5312A1C0
 P 8200 5050
-F 0 "#PWR21" H 8200 5150 30  0001 C CNN
+F 0 "#PWR20" H 8200 5150 30  0001 C CNN
 F 1 "FE_V+" H 8200 5150 30  0000 C CNN
 F 2 "" H 8200 5050 60  0000 C CNN
@@
 $EndComp
 $Comp
-L FE_V- #PWR19
+L FE_V- #PWR18
 U 1 1 5312A1C6
 P 8200 2700
-F 0 "#PWR19" H 8200 2900 40  0001 C CNN
+F 0 "#PWR18" H 8200 2900 40  0001 C CNN
 F 1 "FE_V-" H 8200 2850 40  0000 C CNN
 F 2 "" H 8200 2700 60  0000 C CNN
@@
 $EndComp
 $Comp
-L FE_V+ #PWR18
+L FE_V+ #PWR17
 U 1 1 5312A1D1
 P 8200 1700
-F 0 "#PWR18" H 8200 1800 30  0001 C CNN
+F 0 "#PWR17" H 8200 1800 30  0001 C CNN
 F 1 "FE_V+" H 8200 1800 30  0000 C CNN
 F 2 "" H 8200 1700 60  0000 C CNN
@@
 $EndComp
 $Comp
-L AGND #PWR15
+L AGND #PWR14
 U 1 1 53198D6E
 P 5950 6900
-F 0 "#PWR15" H 5950 6900 40  0001 C CNN
+F 0 "#PWR14" H 5950 6900 40  0001 C CNN
 F 1 "AGND" H 5950 6830 50  0000 C CNN
 F 2 "" H 5950 6900 60  0000 C CNN
@@
 $EndComp
 $Comp
-L AGND #PWR13
+L AGND #PWR12
 U 1 1 53198D7D
 P 5300 4700
-F 0 "#PWR13" H 5300 4700 40  0001 C CNN
+F 0 "#PWR12" H 5300 4700 40  0001 C CNN
 F 1 "AGND" H 5300 4630 50  0000 C CNN
 F 2 "" H 5300 4700 60  0000 C CNN
@@
 $EndComp
 $Comp
-L AGND #PWR12
+L AGND #PWR11
 U 1 1 53198D8C
 P 4550 4200
-F 0 "#PWR12" H 4550 4200 40  0001 C CNN
+F 0 "#PWR11" H 4550 4200 40  0001 C CNN
 F 1 "AGND" H 4550 4130 50  0000 C CNN
 F 2 "" H 4550 4200 60  0000 C CNN
@@
 $EndComp
 $Comp
-L AGND #PWR11
+L AGND #PWR10
 U 1 1 53198D9B
 P 4550 3650
-F 0 "#PWR11" H 4550 3650 40  0001 C CNN
+F 0 "#PWR10" H 4550 3650 40  0001 C CNN
 F 1 "AGND" H 4550 3580 50  0000 C CNN
 F 2 "" H 4550 3650 60  0000 C CNN
@@
 $EndComp
 $Comp
-L AGND #PWR7
+L AGND #PWR6
 U 1 1 53198DAA
 P 2500 5250
-F 0 "#PWR7" H 2500 5250 40  0001 C CNN
+F 0 "#PWR6" H 2500 5250 40  0001 C CNN
 F 1 "AGND" H 2500 5180 50  0000 C CNN
 F 2 "" H 2500 5250 60  0000 C CNN
@@
 $EndComp
 $Comp
-L AGND #PWR9
+L AGND #PWR8
 U 1 1 53198DB9
 P 2950 5250
-F 0 "#PWR9" H 2950 5250 40  0001 C CNN
+F 0 "#PWR8" H 2950 5250 40  0001 C CNN
 F 1 "AGND" H 2950 5180 50  0000 C CNN
 F 2 "" H 2950 5250 60  0000 C CNN
@@
 L AGND #PWR5
 U 1 1 53198DC8
-P 1900 1250
-F 0 "#PWR5" H 1900 1250 40  0001 C CNN
-F 1 "AGND" H 1900 1180 50  0000 C CNN
-F 2 "" H 1900 1250 60  0000 C CNN
-F 3 "" H 1900 1250 60  0000 C CNN
-	1    1900 1250
-	1    0    0    -1
-$EndComp
-$Comp
-L AGND #PWR10
+P 1500 1250
+F 0 "#PWR5" H 1500 1250 40  0001 C CNN
+F 1 "AGND" H 1500 1180 50  0000 C CNN
+F 2 "" H 1500 1250 60  0000 C CNN
+F 3 "" H 1500 1250 60  0000 C CNN
+	1    1500 1250
+	1    0    0    -1
+$EndComp
+$Comp
+L AGND #PWR9
 U 1 1 53198DD7
-P 3550 1250
-F 0 "#PWR10" H 3550 1250 40  0001 C CNN
-F 1 "AGND" H 3550 1180 50  0000 C CNN
-F 2 "" H 3550 1250 60  0000 C CNN
-F 3 "" H 3550 1250 60  0000 C CNN
-	1    3550 1250
-	1    0    0    -1
-$EndComp
-$Comp
-L AGND #PWR23
+P 3750 1250
+F 0 "#PWR9" H 3750 1250 40  0001 C CNN
+F 1 "AGND" H 3750 1180 50  0000 C CNN
+F 2 "" H 3750 1250 60  0000 C CNN
+F 3 "" H 3750 1250 60  0000 C CNN
+	1    3750 1250
+	1    0    0    -1
+$EndComp
+$Comp
+L AGND #PWR22
 U 1 1 53198DE6
 P 9900 6250
-F 0 "#PWR23" H 9900 6250 40  0001 C CNN
+F 0 "#PWR22" H 9900 6250 40  0001 C CNN
 F 1 "AGND" H 9900 6180 50  0000 C CNN
 F 2 "" H 9900 6250 60  0000 C CNN
@@
 $EndComp
 $Comp
-L AGND #PWR25
+L AGND #PWR24
 U 1 1 53198DF5
 P 10250 6250
-F 0 "#PWR25" H 10250 6250 40  0001 C CNN
+F 0 "#PWR24" H 10250 6250 40  0001 C CNN
 F 1 "AGND" H 10250 6180 50  0000 C CNN
 F 2 "" H 10250 6250 60  0000 C CNN
@@
 	1    0    0    -1
 $EndComp
+$Comp
+L INDUCTOR L5
+U 1 1 532400BF
+P 2500 850
+F 0 "L5" V 2450 850 40  0000 C CNN
+F 1 "INDUCTOR" V 2600 850 40  0000 C CNN
+F 2 "SM0805" V 2400 850 60  0000 C CNN
+F 3 "~" H 2500 850 60  0000 C CNN
+	1    2500 850
+	0    1    -1   0
+$EndComp
+Wire Wire Line
+	2950 750  2950 1250
+Wire Wire Line
+	3250 1150 2950 1150
+Connection ~ 2950 1150
+Wire Wire Line
+	2800 850  2950 850
+Connection ~ 2950 850
+Wire Wire Line
+	2000 1150 2500 1150
+Wire Wire Line
+	2500 1150 2500 1250
+Wire Wire Line
+	2200 850  2150 850
+Wire Wire Line
+	2150 850  2150 1150
+Connection ~ 2150 1150
 $EndSCHEMATC

Commit message: Layout v14.0
Parts:
- added C26, C27: C, SM0805, symbol C
Connections:
- net at U2.15 (OSC1): now also C26.1
- net at U2.16 (OSC2): now also C26.2
- net REF+: no longer names the net of U2.9 (REFIN/OUT+)
- net REF+: now also C27.1
- net REF-: no longer names the net of U2.10 (REFIN-)
- net REF-: now also C27.2
Changed lines of the file:
@@
 $EndComp
 $Comp
-L -12V #PWR23
+L -12V #PWR05
 U 1 1 52F4A357
 P 10250 5500
-F 0 "#PWR23" H 10250 5630 20  0001 C CNN
+F 0 "#PWR05" H 10250 5630 20  0001 C CNN
 F 1 "-12V" H 10250 5600 30  0000 C CNN
 F 2 "" H 10250 5500 60  0000 C CNN
@@
 $EndComp
 $Comp
-L +12V #PWR21
+L +12V #PWR06
 U 1 1 52F4A37C
 P 9900 5500
-F 0 "#PWR21" H 9900 5450 20  0001 C CNN
+F 0 "#PWR06" H 9900 5450 20  0001 C CNN
 F 1 "+12V" H 9900 5600 30  0000 C CNN
 F 2 "" H 9900 5500 60  0000 C CNN
@@
 	6050 6800 6050 6650
 $Comp
-L +5V #PWR13
+L +5V #PWR07
 U 1 1 53096E41
 P 5900 5250
-F 0 "#PWR13" H 5900 5340 20  0001 C CNN
+F 0 "#PWR07" H 5900 5340 20  0001 C CNN
 F 1 "+5V" H 5900 5340 30  0000 C CNN
 F 2 "" H 5900 5250 60  0000 C CNN
@@
 	6550 5300 6550 5850
 $Comp
-L +5V #PWR7
+L +5V #PWR08
 U 1 1 53097117
 P 2950 750
-F 0 "#PWR7" H 2950 840 20  0001 C CNN
+F 0 "#PWR08" H 2950 840 20  0001 C CNN
 F 1 "+5V" H 2950 840 30  0000 C CNN
 F 2 "" H 2950 750 60  0000 C CNN
@@
 	1    0    0    -1
 $EndComp
-Text GLabel 4450 1800 2    60   Input ~ 0
-REF+
-Text GLabel 4450 2100 2    60   Input ~ 0
-REF-
 Wire Wire Line
 	4450 1800 4300 1800
@@
 $EndComp
 $Comp
-L FE_V+ #PWR16
+L FE_V+ #PWR09
 U 1 1 5312A1A0
 P 6050 3850
-F 0 "#PWR16" H 6050 3950 30  0001 C CNN
+F 0 "#PWR09" H 6050 3950 30  0001 C CNN
 F 1 "FE_V+" H 6050 3950 30  0000 C CNN
 F 2 "" H 6050 3850 60  0000 C CNN
@@
 $EndComp
 $Comp
-L FE_V+ #PWR20
+L FE_V+ #PWR010
 U 1 1 5312A1C0
 P 8200 5050
-F 0 "#PWR20" H 8200 5150 30  0001 C CNN
+F 0 "#PWR010" H 8200 5150 30  0001 C CNN
 F 1 "FE_V+" H 8200 5150 30  0000 C CNN
 F 2 "" H 8200 5050 60  0000 C CNN
@@
 $EndComp
 $Comp
-L FE_V+ #PWR17
+L FE_V+ #PWR011
 U 1 1 5312A1D1
 P 8200 1700
-F 0 "#PWR17" H 8200 1800 30  0001 C CNN
+F 0 "#PWR011" H 8200 1800 30  0001 C CNN
 F 1 "FE_V+" H 8200 1800 30  0000 C CNN
 F 2 "" H 8200 1700 60  0000 C CNN
@@
 $EndComp
 $Comp
-L AGND #PWR14
+L AGND #PWR012
 U 1 1 53198D6E
 P 5950 6900
-F 0 "#PWR14" H 5950 6900 40  0001 C CNN
+F 0 "#PWR012" H 5950 6900 40  0001 C CNN
 F 1 "AGND" H 5950 6830 50  0000 C CNN
 F 2 "" H 5950 6900 60  0000 C CNN
@@
 $EndComp
 $Comp
-L AGND #PWR12
+L AGND #PWR013
 U 1 1 53198D7D
 P 5300 4700
-F 0 "#PWR12" H 5300 4700 40  0001 C CNN
+F 0 "#PWR013" H 5300 4700 40  0001 C CNN
 F 1 "AGND" H 5300 4630 50  0000 C CNN
 F 2 "" H 5300 4700 60  0000 C CNN
@@
 $EndComp
 $Comp
-L AGND #PWR11
+L AGND #PWR014
 U 1 1 53198D8C
 P 4550 4200
-F 0 "#PWR11" H 4550 4200 40  0001 C CNN
+F 0 "#PWR014" H 4550 4200 40  0001 C CNN
 F 1 "AGND" H 4550 4130 50  0000 C CNN
 F 2 "" H 4550 4200 60  0000 C CNN
@@
 $EndComp
 $Comp
-L AGND #PWR10
+L AGND #PWR015
 U 1 1 53198D9B
 P 4550 3650
-F 0 "#PWR10" H 4550 3650 40  0001 C CNN
+F 0 "#PWR015" H 4550 3650 40  0001 C CNN
 F 1 "AGND" H 4550 3580 50  0000 C CNN
 F 2 "" H 4550 3650 60  0000 C CNN
@@
 $EndComp
 $Comp
-L AGND #PWR6
+L AGND #PWR016
 U 1 1 53198DAA
 P 2500 5250
-F 0 "#PWR6" H 2500 5250 40  0001 C CNN
+F 0 "#PWR016" H 2500 5250 40  0001 C CNN
 F 1 "AGND" H 2500 5180 50  0000 C CNN
 F 2 "" H 2500 5250 60  0000 C CNN
@@
 $EndComp
 $Comp
-L AGND #PWR8
+L AGND #PWR017
 U 1 1 53198DB9
 P 2950 5250
-F 0 "#PWR8" H 2950 5250 40  0001 C CNN
+F 0 "#PWR017" H 2950 5250 40  0001 C CNN
 F 1 "AGND" H 2950 5180 50  0000 C CNN
 F 2 "" H 2950 5250 60  0000 C CNN
@@
 $EndComp
 $Comp
-L AGND #PWR5
+L AGND #PWR018
 U 1 1 53198DC8
 P 1500 1250
-F 0 "#PWR5" H 1500 1250 40  0001 C CNN
+F 0 "#PWR018" H 1500 1250 40  0001 C CNN
 F 1 "AGND" H 1500 1180 50  0000 C CNN
 F 2 "" H 1500 1250 60  0000 C CNN
@@
 $EndComp
 $Comp
-L AGND #PWR9
+L AGND #PWR019
 U 1 1 53198DD7
 P 3750 1250
-F 0 "#PWR9" H 3750 1250 40  0001 C CNN
+F 0 "#PWR019" H 3750 1250 40  0001 C CNN
 F 1 "AGND" H 3750 1180 50  0000 C CNN
 F 2 "" H 3750 1250 60  0000 C CNN
@@
 $EndComp
 $Comp
-L AGND #PWR22
+L AGND #PWR020
 U 1 1 53198DE6
 P 9900 6250
-F 0 "#PWR22" H 9900 6250 40  0001 C CNN
+F 0 "#PWR020" H 9900 6250 40  0001 C CNN
 F 1 "AGND" H 9900 6180 50  0000 C CNN
 F 2 "" H 9900 6250 60  0000 C CNN
@@
 $EndComp
 $Comp
-L AGND #PWR24
+L AGND #PWR021
 U 1 1 53198DF5
 P 10250 6250
-F 0 "#PWR24" H 10250 6250 40  0001 C CNN
+F 0 "#PWR021" H 10250 6250 40  0001 C CNN
 F 1 "AGND" H 10250 6180 50  0000 C CNN
 F 2 "" H 10250 6250 60  0000 C CNN
@@
 	2150 850  2150 1150
 Connection ~ 2150 1150
+$Comp
+L C C26
+U 1 1 532691CB
+P 1150 1950
+F 0 "C26" H 1150 2050 40  0000 L CNN
+F 1 "C" H 1156 1865 40  0000 L CNN
+F 2 "SM0805" H 1188 1800 30  0000 C CNN
+F 3 "~" H 1150 1950 60  0000 C CNN
+	1    1150 1950
+	1    0    0    -1
+$EndComp
+Wire Wire Line
+	1150 1750 1150 1600
+Wire Wire Line
+	1150 1600 1400 1600
+Wire Wire Line
+	1400 1600 1400 1800
+Wire Wire Line
+	1150 2150 1150 2250
+Wire Wire Line
+	1150 2250 1400 2250
+Wire Wire Line
+	1400 2250 1400 2050
+$Comp
+L C C27
+U 1 1 532692C1
+P 4650 1950
+F 0 "C27" H 4650 2050 40  0000 L CNN
+F 1 "C" H 4656 1865 40  0000 L CNN
+F 2 "SM0805" H 4688 1800 30  0000 C CNN
+F 3 "~" H 4650 1950 60  0000 C CNN
+	1    4650 1950
+	1    0    0    -1
+$EndComp
+Wire Wire Line
+	4650 1750 4650 1600
+Wire Wire Line
+	4650 1600 4450 1600
+Wire Wire Line
+	4450 1600 4450 1800
+Wire Wire Line
+	4450 2100 4450 2300
+Wire Wire Line
+	4450 2300 4650 2300
+Wire Wire Line
+	4650 2300 4650 2150
 $EndSCHEMATC

Commit message: Layout v16.0
Parts:
- added TP2: +5V, symbol CONN_1
- added TP3: CH0+, symbol CONN_1
- added TP4: CH1+, symbol CONN_1
Connections:
- net +5V: now also TP2.1
- net at C8.1, R23.1, U2.4 (CH0+)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: now also TP3.1
- net at U2.7 (CH1+), U3.3 (OUT): now also TP4.1
Changed lines of the file:
@@
 Sheet 3 9
 Title ""
-Date "17 mar 2014"
+Date "22 mar 2014"
 Rev ""
 Comp ""
@@
 Wire Wire Line
 	4650 2300 4650 2150
+$Comp
+L CONN_1 TP3
+U 1 1 532D4A9C
+P 4550 3100
+F 0 "TP3" H 4630 3100 40  0000 L CNN
+F 1 "CH0+" H 4550 3155 30  0001 C CNN
+F 2 "" H 4550 3100 60  0000 C CNN
+F 3 "" H 4550 3100 60  0000 C CNN
+	1    4550 3100
+	0    -1   -1   0
+$EndComp
+$Comp
+L CONN_1 TP4
+U 1 1 532D4ABD
+P 4850 3750
+F 0 "TP4" H 4930 3750 40  0000 L CNN
+F 1 "CH1+" H 4850 3805 30  0001 C CNN
+F 2 "" H 4850 3750 60  0000 C CNN
+F 3 "" H 4850 3750 60  0000 C CNN
+	1    4850 3750
+	0    -1   -1   0
+$EndComp
+$Comp
+L CONN_1 TP2
+U 1 1 532D56D9
+P 3100 700
+F 0 "TP2" H 3180 700 40  0000 L CNN
+F 1 "+5V" H 3100 755 30  0001 C CNN
+F 2 "" H 3100 700 60  0000 C CNN
+F 3 "" H 3100 700 60  0000 C CNN
+	1    3100 700
+	0    -1   -1   0
+$EndComp
+Wire Wire Line
+	3100 850  3100 1150
+Connection ~ 3100 1150
+Wire Wire Line
+	4550 3250 4550 3350
+Connection ~ 4550 3350
 $EndSCHEMATC

Commit message: Layout v17.0
Parts:
- added R53, R54: 1k, ~, symbol R
Connections:
- net AGND: now also R53.1
- net TC_IN_+: now also U4.12 (+); no longer U4.10 (+)
- net TC_IN_-: now also U4.10 (+); no longer U4.12 (+)
- net at TP4.1, U2.7 (CH1+): now also R53.2, R54.1; no longer U3.3 (OUT)
- new net: R54.2, U3.3 (OUT)
Other:
- moved on the sheet: TP4
Changed lines of the file:
@@
 Sheet 3 9
 Title ""
-Date "22 mar 2014"
+Date "23 mar 2014"
 Rev ""
 Comp ""
@@
 $EndDescr
 Text HLabel 8950 2100 2    60   Input ~ 0
+TC_IN_-
+Text HLabel 8950 4650 2    60   Input ~ 0
 TC_IN_+
-Text HLabel 8950 4650 2    60   Input ~ 0
-TC_IN_-
 Text HLabel 1050 3400 0    60   Input ~ 0
 MOSI
@@
 $EndComp
 $Comp
-L -12V #PWR05
+L -12V #PWR23
 U 1 1 52F4A357
 P 10250 5500
-F 0 "#PWR05" H 10250 5630 20  0001 C CNN
+F 0 "#PWR23" H 10250 5630 20  0001 C CNN
 F 1 "-12V" H 10250 5600 30  0000 C CNN
 F 2 "" H 10250 5500 60  0000 C CNN
@@
 $EndComp
 $Comp
-L +12V #PWR06
+L +12V #PWR21
 U 1 1 52F4A37C
 P 9900 5500
-F 0 "#PWR06" H 9900 5450 20  0001 C CNN
+F 0 "#PWR21" H 9900 5450 20  0001 C CNN
 F 1 "+12V" H 9900 5600 30  0000 C CNN
 F 2 "" H 9900 5500 60  0000 C CNN
@@
 	4550 4200 4550 4050
 Wire Wire Line
-	4300 3900 4850 3900
-Wire Wire Line
-	4850 3900 4850 6000
-Wire Wire Line
-	4850 6000 5350 6000
+	4300 3900 4700 3900
+Wire Wire Line
+	4700 3900 4700 6100
 Wire Wire Line
 	5950 6650 5950 6900
@@
 	5850 6650 5850 6800
 Wire Wire Line
-	5850 6800 6550 6800
+	4700 6800 6550 6800
 Connection ~ 5950 6800
 Wire Wire Line
 	6050 6800 6050 6650
 $Comp
-L +5V #PWR07
+L +5V #PWR13
 U 1 1 53096E41
 P 5900 5250
-F 0 "#PWR07" H 5900 5340 20  0001 C CNN
+F 0 "#PWR13" H 5900 5340 20  0001 C CNN
 F 1 "+5V" H 5900 5340 30  0000 C CNN
 F 2 "" H 5900 5250 60  0000 C CNN
@@
 	6550 5300 6550 5850
 $Comp
-L +5V #PWR08
+L +5V #PWR7
 U 1 1 53097117
 P 2950 750
-F 0 "#PWR08" H 2950 840 20  0001 C CNN
+F 0 "#PWR7" H 2950 840 20  0001 C CNN
 F 1 "+5V" H 2950 840 30  0000 C CNN
 F 2 "" H 2950 750 60  0000 C CNN
@@
 $EndComp
 $Comp
-L FE_V+ #PWR09
+L FE_V+ #PWR16
 U 1 1 5312A1A0
 P 6050 3850
-F 0 "#PWR09" H 6050 3950 30  0001 C CNN
+F 0 "#PWR16" H 6050 3950 30  0001 C CNN
 F 1 "FE_V+" H 6050 3950 30  0000 C CNN
 F 2 "" H 6050 3850 60  0000 C CNN
@@
 $EndComp
 $Comp
-L FE_V+ #PWR010
+L FE_V+ #PWR20
 U 1 1 5312A1C0
 P 8200 5050
-F 0 "#PWR010" H 8200 5150 30  0001 C CNN
+F 0 "#PWR20" H 8200 5150 30  0001 C CNN
 F 1 "FE_V+" H 8200 5150 30  0000 C CNN
 F 2 "" H 8200 5050 60  0000 C CNN
@@
 $EndComp
 $Comp
-L FE_V+ #PWR011
+L FE_V+ #PWR17
 U 1 1 5312A1D1
 P 8200 1700
-F 0 "#PWR011" H 8200 1800 30  0001 C CNN
+F 0 "#PWR17" H 8200 1800 30  0001 C CNN
 F 1 "FE_V+" H 8200 1800 30  0000 C CNN
 F 2 "" H 8200 1700 60  0000 C CNN
@@
 $EndComp
 $Comp
-L AGND #PWR012
+L AGND #PWR14
 U 1 1 53198D6E
 P 5950 6900
-F 0 "#PWR012" H 5950 6900 40  0001 C CNN
+F 0 "#PWR14" H 5950 6900 40  0001 C CNN
 F 1 "AGND" H 5950 6830 50  0000 C CNN
 F 2 "" H 5950 6900 60  0000 C CNN
@@
 $EndComp
 $Comp
-L AGND #PWR013
+L AGND #PWR12
 U 1 1 53198D7D
 P 5300 4700
-F 0 "#PWR013" H 5300 4700 40  0001 C CNN
+F 0 "#PWR12" H 5300 4700 40  0001 C CNN
 F 1 "AGND" H 5300 4630 50  0000 C CNN
 F 2 "" H 5300 4700 60  0000 C CNN
@@
 $EndComp
 $Comp
-L AGND #PWR014
+L AGND #PWR11
 U 1 1 53198D8C
 P 4550 4200
-F 0 "#PWR014" H 4550 4200 40  0001 C CNN
+F 0 "#PWR11" H 4550 4200 40  0001 C CNN
 F 1 "AGND" H 4550 4130 50  0000 C CNN
 F 2 "" H 4550 4200 60  0000 C CNN
@@
 $EndComp
 $Comp
-L AGND #PWR015
+L AGND #PWR10
 U 1 1 53198D9B
 P 4550 3650
-F 0 "#PWR015" H 4550 3650 40  0001 C CNN
+F 0 "#PWR10" H 4550 3650 40  0001 C CNN
 F 1 "AGND" H 4550 3580 50  0000 C CNN
 F 2 "" H 4550 3650 60  0000 C CNN
@@
 $EndComp
 $Comp
-L AGND #PWR016
+L AGND #PWR6
 U 1 1 53198DAA
 P 2500 5250
-F 0 "#PWR016" H 2500 5250 40  0001 C CNN
+F 0 "#PWR6" H 2500 5250 40  0001 C CNN
 F 1 "AGND" H 2500 5180 50  0000 C CNN
 F 2 "" H 2500 5250 60  0000 C CNN
@@
 $EndComp
 $Comp
-L AGND #PWR017
+L AGND #PWR8
 U 1 1 53198DB9
 P 2950 5250
-F 0 "#PWR017" H 2950 5250 40  0001 C CNN
+F 0 "#PWR8" H 2950 5250 40  0001 C CNN
 F 1 "AGND" H 2950 5180 50  0000 C CNN
 F 2 "" H 2950 5250 60  0000 C CNN
@@
 $EndComp
 $Comp
-L AGND #PWR018
+L AGND #PWR5
 U 1 1 53198DC8
 P 1500 1250
-F 0 "#PWR018" H 1500 1250 40  0001 C CNN
+F 0 "#PWR5" H 1500 1250 40  0001 C CNN
 F 1 "AGND" H 1500 1180 50  0000 C CNN
 F 2 "" H 1500 1250 60  0000 C CNN
@@
 $EndComp
 $Comp
-L AGND #PWR019
+L AGND #PWR9
 U 1 1 53198DD7
 P 3750 1250
-F 0 "#PWR019" H 3750 1250 40  0001 C CNN
+F 0 "#PWR9" H 3750 1250 40  0001 C CNN
 F 1 "AGND" H 3750 1180 50  0000 C CNN
 F 2 "" H 3750 1250 60  0000 C CNN
@@
 $EndComp
 $Comp
-L AGND #PWR020
+L AGND #PWR22
 U 1 1 53198DE6
 P 9900 6250
-F 0 "#PWR020" H 9900 6250 40  0001 C CNN
+F 0 "#PWR22" H 9900 6250 40  0001 C CNN
 F 1 "AGND" H 9900 6180 50  0000 C CNN
 F 2 "" H 9900 6250 60  0000 C CNN
@@
 $EndComp
 $Comp
-L AGND #PWR021
+L AGND #PWR24
 U 1 1 53198DF5
 P 10250 6250
-F 0 "#PWR021" H 10250 6250 40  0001 C CNN
+F 0 "#PWR24" H 10250 6250 40  0001 C CNN
 F 1 "AGND" H 10250 6180 50  0000 C CNN
 F 2 "" H 10250 6250 60  0000 C CNN
@@
 	2950 750  2950 1250
 Wire Wire Line
-	3250 1150 2950 1150
+	2950 1150 3250 1150
 Connection ~ 2950 1150
 Wire Wire Line
@@
 L CONN_1 TP4
 U 1 1 532D4ABD
-P 4850 3750
-F 0 "TP4" H 4930 3750 40  0000 L CNN
-F 1 "CH1+" H 4850 3805 30  0001 C CNN
-F 2 "" H 4850 3750 60  0000 C CNN
-F 3 "" H 4850 3750 60  0000 C CNN
-	1    4850 3750
+P 4700 3750
+F 0 "TP4" H 4780 3750 40  0000 L CNN
+F 1 "CH1+" H 4700 3805 30  0001 C CNN
+F 2 "" H 4700 3750 60  0000 C CNN
+F 3 "" H 4700 3750 60  0000 C CNN
+	1    4700 3750
 	0    -1   -1   0
 $EndComp
@@
 	4550 3250 4550 3350
 Connection ~ 4550 3350
+$Comp
+L R R54
+U 1 1 532E99C8
+P 5050 6000
+F 0 "R54" V 5130 6000 40  0000 C CNN
+F 1 "1k" V 5057 6001 40  0000 C CNN
+F 2 "~" V 4980 6000 30  0000 C CNN
+F 3 "~" H 5050 6000 30  0000 C CNN
+	1    5050 6000
+	0    -1   -1   0
+$EndComp
+Wire Wire Line
+	5300 6000 5350 6000
+Wire Wire Line
+	4700 6000 4800 6000
+$Comp
+L R R53
+U 1 1 532E9AFB
+P 4700 6350
+F 0 "R53" V 4780 6350 40  0000 C CNN
+F 1 "1k" V 4707 6351 40  0000 C CNN
+F 2 "~" V 4630 6350 30  0000 C CNN
+F 3 "~" H 4700 6350 30  0000 C CNN
+	1    4700 6350
+	-1   0    0    1
+$EndComp
+Connection ~ 4700 6000
+Wire Wire Line
+	4700 6600 4700 6800
+Connection ~ 5850 6800
 $EndSCHEMATC
